Commit message: Add first version of climbing robot urdf

File: robots/climbingrobot.urdf.xacro (robot description, xacro)
@@ -1,30 +1,447 @@
 <?xml version="1.0" ?>
-<robot name="climbingrobot" xmlns:xacro="http://ros.org/wiki/xacro">
-    <!--- new_gazebo_version should be false by default because pinocchio needs it!-->
-    <xacro:arg name="robot_name" default="climbingrobot"/>
-    <xacro:arg name="new_gazebo_version" default="false"/>
-    <xacro:include filename="$(find climbingrobot_description)/gazebo/gazebo.urdf.xacro">
-        <xacro:arg name="task_period" value="$(arg task_period)"/>
-	<xacro:arg name="robot_name" value="$(arg robot_name)"/>
-    </xacro:include>
-    <!-- BASE LINK -->
-    <!-- floating type is supported in older versions of Gazebo. In new Gazebo if a link has no parent, it is supposed to be attached to a floating joint -->
-    <xacro:unless value="$(arg new_gazebo_version)">
-        <!-- Floating-base Joint -->
-        <link name="world"/>
-        <joint name="floating_base_joint" type="floating" >
-            <origin rpy="0 0 0" xyz="0 0 0"/>
-            <parent link="world"/>
-            <child link="base_link"/>
-        </joint>
-    </xacro:unless>
-    <link name="base_link" />
-    <joint name="floating_base" type="fixed">
-        <origin rpy="0 0 0" xyz="0 0 0"/>
-        <parent link="base_link"/>
-        <child link="trunk"/>
-    </joint>
-    <link name="trunk">
-        <!-- TODO the trunk (it will be fixed to base link but it has inertia) -->
-    </link>
+<robot name="climber">
+  <!-- This file is based on: https://atlas.is.localnet/confluence/display/AMDW/Quadruped+URDF+Files -->
+  <link name="mountain">
+    <!--<visual>
+      <origin rpy="0 0 0" xyz="0 0 0"/>
+      <geometry>
+        <mesh filename="package://model/urdf/meshes/obj/cube.obj" scale="0.01 10.0 10.0"/>
+      </geometry>
+      <material name="ground">
+        <color rgba=".9 .1 .1 .5"/>
+      </material>
+    </visual>-->
+    <collision>
+      <origin rpy="0 0 0" xyz="0 0 0.0"/>
+      <geometry>
+        <box size="0.1 10.0 10.0"/>
+      </geometry>
+    </collision>
+    <inertial>
+      <origin rpy="0 0 0" xyz="0 0 0.0"/>
+      <mass value="1000.0"/>
+      <inertia ixx="10.0" ixy="0.0" ixz="0.0" iyy="10.0" iyz="0.0" izz="10.0"/>
+    </inertial>
+  </link>
+  <!-- Revolute pitch joint between the mountain and the wire -->
+  <joint name="mountain_wire_pitch" type="revolute">
+    <parent link="mountain"/>
+    <child link="pre-wire1"/>
+    <limit effort="3" lower="-10" upper="10" velocity="1000"/>
+    <!-- joint rotates about y axis -->
+    <axis xyz="0 1 0"/>
+    <origin rpy="0 0 0" xyz="0.0 0.0 0.0"/>
+    <!-- pybullet simulation parameters -->
+    <dynamics damping="0.0" friction="0.0"/>
+  </joint>
+  <link name="pre-wire1">
+    <visual>
+      <origin rpy="0 0 0" xyz="0 0 0"/>
+      <geometry>
+        <mesh filename="package://model/urdf/meshes/obj/cylinder.obj" scale="0.01 0.01 0.01"/>
+      </geometry>
+      <material name="grey">
+        <color rgba=".7 .7 .7 .5"/>
+      </material>
+    </visual>
+    <collision>
+      <origin rpy="0 0 0" xyz="0 0 0.0"/>
+      <geometry>
+        <cylinder length="0.01" radius="0.01"/>
+      </geometry>
+    </collision>
+    <inertial>
+      <origin rpy="0 0 0" xyz="0 0 0.0"/>
+      <mass value="0.01"/>
+      <inertia ixx="0.0001" ixy="0.0" ixz="0.0" iyy="0.0001" iyz="0.0" izz="0.0001"/>
+    </inertial>
+  </link>
+  <!-- Revolute roll joint between the mountain and the wire -->
+  <joint name="mountain_wire_roll" type="revolute">
+    <parent link="pre-wire1"/>
+    <child link="pre-wire2"/>
+    <limit effort="3" lower="-10" upper="10" velocity="1000"/>
+    <!-- joint rotates about x axis -->
+    <axis xyz="1 0 0"/>
+    <origin rpy="0 0 0" xyz="0.0 0.0 0.0"/>
+    <!-- pybullet simulation parameters -->
+    <dynamics damping="0.0" friction="0.0"/>
+  </joint>
+  <link name="pre-wire2">
+    <visual>
+      <origin rpy="0 0 0" xyz="0 0 0"/>
+      <geometry>
+        <mesh filename="package://model/urdf/meshes/obj/cylinder.obj" scale="0.01 0.01 0.01"/>
+      </geometry>
+      <material name="grey">
+        <color rgba=".7 .7 .7 .5"/>
+      </material>
+    </visual>
+    <collision>
+      <origin rpy="0 0 0" xyz="0 0 0.0"/>
+      <geometry>
+        <cylinder length="0.01" radius="0.01"/>
+      </geometry>
+    </collision>
+    <inertial>
+      <origin rpy="0 0 0" xyz="0 0 0.0"/>
+      <mass value="0.01"/>
+      <inertia ixx="0.0001" ixy="0.0" ixz="0.0" iyy="0.0001" iyz="0.0" izz="0.0001"/>
+    </inertial>
+  </link>
+  <!-- Revolute yaw joint between the mountain and the wire -->
+  <joint name="mountain_wire_yaw" type="revolute">
+    <parent link="pre-wire2"/>
+    <child link="wire"/>
+    <limit effort="3" lower="-10" upper="10" velocity="1000"/>
+    <!-- joint rotates about z axis -->
+    <axis xyz="0 0 1"/>
+    <origin rpy="0 0 0" xyz="0.0 0.0 0.0"/>
+    <!-- pybullet simulation parameters -->
+    <dynamics damping="0.0" friction="0.0"/>
+  </joint>
+  <link name="wire">
+    <visual>
+      <origin rpy="0 0 0" xyz="0 0 -2"/>
+      <geometry>
+        <mesh filename="package://model/urdf/meshes/obj/cylinder.obj" scale="0.01 0.01 4.0"/>
+      </geometry>
+      <material name="grey">
+        <color rgba=".7 .7 .7 .5"/>
+      </material>
+    </visual>
+    <collision>
+      <origin rpy="0 0 0" xyz="0 0 0.0"/>
+      <geometry>
+        <cylinder length="4" radius="0.01"/>
+      </geometry>
+    </collision>
+    <inertial>
+      <origin rpy="0 0 0" xyz="0 0 0.0"/>
+      <mass value="0.01"/>
+      <inertia ixx="0.0001" ixy="0.0" ixz="0.0" iyy="0.0001" iyz="0.0" izz="1e-6"/>
+    </inertial>
+  </link>
+  <!-- Prismatic joint between the wire and the base -->
+  <joint name="wire_base_prismatic" type="prismatic">
+    <parent link="wire"/>
+    <child link="pre-base1"/>
+    <limit effort="3" lower="-10" upper="10" velocity="1000"/>
+    <!-- joint translates on x axis -->
+    <axis xyz="0 0 1"/>
+    <origin rpy="0 0 0" xyz="0.0 0.0 -2.0"/>
+    <!-- pybullet simulation parameters -->
+    <dynamics damping="0.0" friction="0.0"/>
+  </joint>
+  <link name="pre-base1">
+    <visual>
+      <origin rpy="0 0 0" xyz="0 0 0"/>
+      <geometry>
+        <mesh filename="package://model/urdf/meshes/obj/cylinder.obj" scale="0.01 0.01 0.01"/>
+      </geometry>
+      <material name="grey">
+        <color rgba=".7 .7 .7 .5"/>
+      </material>
+    </visual>
+    <collision>
+      <origin rpy="0 0 0" xyz="0 0 0.0"/>
+      <geometry>
+        <cylinder length="0.01" radius="0.01"/>
+      </geometry>
+    </collision>
+    <inertial>
+      <origin rpy="0 0 0" xyz="0 0 0.0"/>
+      <mass value="0.01"/>
+      <inertia ixx="0.0001" ixy="0.0" ixz="0.0" iyy="0.0001" iyz="0.0" izz="0.0001"/>
+    </inertial>
+  </link>
+  <!-- Revolute pitch joint between the wire and the base -->
+  <joint name="wire_base_pitch" type="revolute">
+    <parent link="pre-base1"/>
+    <child link="pre-base2"/>
+    <limit effort="3" lower="-10" upper="10" velocity="1000"/>
+    <!-- joint rotates about y axis -->
+    <axis xyz="0 1 0"/>
+    <origin rpy="0 0 0" xyz="0.0 0.0 0.0"/>
+    <!-- pybullet simulation parameters -->
+    <dynamics damping="0.0" friction="0.0"/>
+  </joint>
+  <link name="pre-base2">
+    <visual>
+      <origin rpy="0 0 0" xyz="0 0 0"/>
+      <geometry>
+        <mesh filename="package://model/urdf/meshes/obj/cylinder.obj" scale="0.01 0.01 0.01"/>
+      </geometry>
+      <material name="grey">
+        <color rgba=".7 .7 .7 .5"/>
+      </material>
+    </visual>
+    <collision>
+      <origin rpy="0 0 0" xyz="0 0 0.0"/>
+      <geometry>
+        <cylinder length="0.01" radius="0.01"/>
+      </geometry>
+    </collision>
+    <inertial>
+      <origin rpy="0 0 0" xyz="0 0 0.0"/>
+      <mass value="0.01"/>
+      <inertia ixx="0.0001" ixy="0.0" ixz="0.0" iyy="0.0001" iyz="0.0" izz="0.0001"/>
+    </inertial>
+  </link>
+  <!-- Revolute roll joint between the wire and the base -->
+  <joint name="wire_base_roll" type="revolute">
+    <parent link="pre-base2"/>
+    <child link="pre-base3"/>
+    <limit effort="3" lower="-10" upper="10" velocity="1000"/>
+    <!-- joint rotates about x axis -->
+    <axis xyz="1 0 0"/>
+    <origin rpy="0 0 0" xyz="0.0 0.0 0.0"/>
+    <!-- pybullet simulation parameters -->
+    <dynamics damping="0.0" friction="0.0"/>
+  </joint>
+  <link name="pre-base3">
+    <visual>
+      <origin rpy="0 0 0" xyz="0 0 0"/>
+      <geometry>
+        <mesh filename="package://model/urdf/meshes/obj/cylinder.obj" scale="0.01 0.01 0.01"/>
+      </geometry>
+      <material name="grey">
+        <color rgba=".7 .7 .7 .5"/>
+      </material>
+    </visual>
+    <collision>
+      <origin rpy="0 0 0" xyz="0 0 0.0"/>
+      <geometry>
+        <cylinder length="0.01" radius="0.01"/>
+      </geometry>
+    </collision>
+    <inertial>
+      <origin rpy="0 0 0" xyz="0 0 0.0"/>
+      <mass value="0.01"/>
+      <inertia ixx="0.0001" ixy="0.0" ixz="0.0" iyy="0.0001" iyz="0.0" izz="0.0001"/>
+    </inertial>
+  </link>
+  <!-- Revolute yaw joint between the wire and the base -->
+  <joint name="wire_base_yaw" type="revolute">
+    <parent link="pre-base3"/>
+    <child link="base"/>
+    <limit effort="3" lower="-10" upper="10" velocity="1000"/>
+    <!-- joint rotates about z axis -->
+    <axis xyz="0 0 1"/>
+    <origin rpy="0 0 0" xyz="0.0 0.0 0.0"/>
+    <!-- pybullet simulation parameters -->
+    <dynamics damping="0.0" friction="0.0"/>
+  </joint>
+  <link name="base">
+    <!-- BASE LINK INERTIAL -->
+    <inertial>
+      <origin rpy="0 0 0" xyz="0 0 0"/>
+      <!-- <mass value="0.36"/> -->
+      <mass value="1.0"/>
+      <!-- The base is extremely symmetrical. -->
+      <inertia ixx="1.0" ixy="0.0" ixz="0.0" iyy="1.0" iyz="0.0" izz="1.0"/>
+    </inertial>
+    <!-- BASE LINK VISUAL -->
+    <visual>
+      <origin rpy="0 0 0" xyz="0 0 0"/>
+      <geometry>
+        <mesh filename="package://model/urdf/meshes/obj/with_foot/solo_body.obj" scale="1 1 1"/>
+      </geometry>
+      <material name="red">
+        <color rgba="0.749 0.380 0.410 1.0"/>
+      </material>
+    </visual>
+    <!-- BASE LINK COLLISION -->
+    <collision>
+      <origin rpy="0 0 0" xyz="0 0 0"/>
+      <geometry>
+        <mesh filename="package://model/urdf/meshes/obj/with_foot/solo_body.obj" scale="1 1 1"/>
+      </geometry>
+    </collision>
+    <!-- Bullet specific paramters -->
+    <contact>
+      <lateral_friction value="1.0"/>
+      <restitution value="0.5"/>
+    </contact>
+  </link>
+  <!-- END BASE LINK -->
+  <!-- Joint between the base and the ${prefix} upper leg -->
+  <joint name="hip_pitch" type="revolute">
+    <parent link="base"/>
+    <child link="upper_link1"/>
+    <limit effort="3" lower="-10" upper="10" velocity="1000"/>
+    <!-- joints rotates around the y-axis -->
+    <axis xyz="0 1 0"/>
+    <origin rpy="0 0 0" xyz="0.0 -0.02 0.025"/>
+    <!-- pybullet simulation parameters -->
+    <dynamics damping="0.0" friction="0.0"/>
+  </joint>
+  <link name="upper_link1">
+    <!-- Left upper leg inertia -->
+    <inertial>
+      <origin rpy="0 0 0" xyz="0.0000 0.0 -0.0"/>
+      <mass value="0.01"/>
+      <inertia ixx="0.00041107" ixy="0.0" ixz="0.0" iyy="0.00041193" iyz="0.00004671" izz="0.00003024"/>
+    </inertial>
+    <!-- UPPER LEG LINK VISUAL
+    <visual>
+      <origin rpy="0 0 0" xyz="0 0 0"/>
+      <geometry>
+        <mesh filename="package://model/urdf/meshes/obj/with_foot/solo_upper_leg_left_side.obj"/>
+      </geometry>
+      <material name="grey">
+        <color rgba="0.8 0.8 0.8 1.0"/>
+      </material>
+    </visual>-->
+    <!-- UPPER LEG LINK COLLISION
+    <collision>
+      <origin rpy="0 0 0" xyz="0 0 0"/>
+      <geometry>
+        <mesh filename="package://model/urdf/meshes/obj/with_foot/solo_upper_leg_left_side.obj"/>
+      </geometry>
+        <material name="white">
+        	<color rgba="0.898 0.913 0.941 1.0"/>
+    	</material>
+    </collision>-->
+    <!-- Bullet specific paramters -->
+    <contact>
+      <lateral_friction value="1.0"/>
+      <restitution value="0.5"/>
+    </contact>
+  </link>
+  <joint name="hip_roll" type="revolute">
+    <parent link="upper_link1"/>
+    <child link="upper_link2"/>
+    <limit effort="3" lower="-10" upper="10" velocity="1000"/>
+    <!-- joints rotates around the y-axis -->
+    <axis xyz="1 0 0"/>
+    <origin rpy="0 0 0" xyz="0.0 0.0 0.0"/>
+    <!-- pybullet simulation parameters -->
+    <dynamics damping="0.0" friction="0.0"/>
+  </joint>
+  <link name="upper_link2">
+    <!-- Left upper leg inertia -->
+    <inertial>
+      <origin rpy="0 0 0" xyz="0.0000 0.0 -0.0"/>
+      <mass value="0.14853845"/>
+      <inertia ixx="0.00041107" ixy="0.0" ixz="0.0" iyy="0.00041193" iyz="0.00004671" izz="0.00003024"/>
+    </inertial>
+    <!-- UPPER LEG LINK VISUAL -->
+    <visual>
+      <origin rpy="0 0 0" xyz="0 0 0"/>
+      <geometry>
+        <mesh filename="package://model/urdf/meshes/obj/with_foot/solo_upper_leg_left_side.obj"/>
+      </geometry>
+      <material name="grey">
+        <color rgba="0.7 0.7 0.7 0.5"/>
+      </material>
+    </visual>
+    <!-- UPPER LEG LINK COLLISION -->
+    <collision>
+      <origin rpy="0 0 0" xyz="0 0 0"/>
+      <geometry>
+        <mesh filename="package://model/urdf/meshes/obj/with_foot/solo_upper_leg_left_side.obj"/>
+      </geometry>
+        <material name="white">
+        	<color rgba="0.898 0.913 0.941 1.0"/>
+    	</material>
+    </collision>
+    <!-- Bullet specific paramters -->
+    <contact>
+      <lateral_friction value="1.0"/>
+      <restitution value="0.5"/>
+    </contact>
+  </link>
+  <!-- END UPPER LEG LINK -->
+  <!-- KFE: Joint between the upper leg and the lower leg -->
+  <joint name="knee" type="prismatic">
+    <parent link="upper_link2"/>
+    <child link="lower_link"/>
+    <limit effort="3" lower="-10" upper="10" velocity="1000"/>
+    <!-- joints rotates around the y-axis -->
+    <axis xyz="0 0 1"/>
+    <origin rpy="0 0 0" xyz="0 0.02 -0.08"/>
+    <!-- pybullet simulation parameters -->
+    <dynamics damping="0.0" friction="0.0"/>
+  </joint>
+  <link name="lower_link">
+    <!-- Left lower leg inertia -->
+    <inertial>
+      <origin rpy="0 0 0" xyz="0.0 0.0 -0.09"/>
+      <mass value="0.0307"/>
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