Commit message: works without leg

File: urdf/climbingrobot.transmission.xacro (robot description, xacro)
@@ -2,34 +2,4 @@
 <robot xmlns:xacro="http://ros.org/wiki/xacro">
         <xacro:macro name="climbingrobot_transmission">
-		<transmission name="anchor_x_joint">
-                        <type>transmission_interface/SimpleTransmission</type>
-                        <joint name="anchor_x_joint">
-                                <hardwareInterface>hardware_interface/EffortJointInterface</hardwareInterface>
-                        </joint>
-                        <actuator name="anchor_x_joint">
-                                <hardwareInterface>hardware_interface/EffortJointInterface</hardwareInterface>
-                                <mechanicalReduction>1</mechanicalReduction>
-                        </actuator>
-                </transmission>
-		<transmission name="anchor_y_joint">
-                        <type>transmission_interface/SimpleTransmission</type>
-                        <joint name="anchor_y_joint">
-                                <hardwareInterface>hardware_interface/EffortJointInterface</hardwareInterface>
-                        </joint>
-                        <actuator name="anchor_y_joint">
-                                <hardwareInterface>hardware_interface/EffortJointInterface</hardwareInterface>
-                                <mechanicalReduction>1</mechanicalReduction>
-                        </actuator>
-                </transmission>
-		<transmission name="anchor_z_joint">
-                        <type>transmission_interface/SimpleTransmission</type>
-                        <joint name="anchor_z_joint">
-                                <hardwareInterface>hardware_interface/EffortJointInterface</hardwareInterface>
-                        </joint>
-                        <actuator name="anchor_z_joint">
-                                <hardwareInterface>hardware_interface/EffortJointInterface</hardwareInterface>
-                                <mechanicalReduction>1</mechanicalReduction>
-                        </actuator>
-                </transmission>
   		<transmission name="mountain_wire_pitch">
                         <type>transmission_interface/SimpleTransmission</type>

File: urdf/climbingrobot.xacro (robot description, xacro)
@@ -11,36 +11,8 @@
     <xacro:include filename="$(find climbingrobot_description)/urdf/climbingrobot.transmission.xacro"/>
     <link name="world"/>
-    <joint name="anchor_x_joint" type="prismatic">
-	<parent link="world"/>
-	<child link="fake_link1"/>
-	<axis xyz="1 0 0 "/>
-	<origin xyz="0 0 0" rpy="0 0 0"/>
-	<limit effort="1000" velocity="100.0" lower="-100" upper="100"/>
-    </joint>
-    <link name="fake_link1">
-	<inertial>
-	<mass value="0.00001"/>
-	<inertia ixx="5.8083e-4" ixy="0" ixz="0" iyy="3.0833e-5" iyz="0" izz="5.9083e-4"/>
-	</inertial>
-    </link>
-    <joint name="anchor_y_joint" type="prismatic">
-		<parent link="fake_link1"/>
-		<child link="fake_link2"/>
-		<axis xyz="0 1 0 "/>
-		<origin xyz="0 0 0" rpy="0 0 0"/>
-		<limit effort="1000" velocity="100.0" lower="-100" upper="100"/>
-    </joint>
-    <link name="fake_link2">
-	<inertial>
-	<mass value="0.00001"/>
-	<inertia ixx="5.8083e-4" ixy="0" ixz="0" iyy="3.0833e-5" iyz="0" izz="5.9083e-4"/>
-	</inertial>
-    </link>
-    <joint name="anchor_z_joint" type="prismatic">
-		<parent link="fake_link2"/>
-		<child link="anchor"/>
-		<axis xyz="0 0 1 "/>
-		<origin xyz="0 0 0" rpy="0 0 0"/>
-		<limit effort="1000" velocity="100.0" lower="-100" upper="100"/>
+   <joint name="mountain" type="fixed">
+        <origin rpy="0 0 0" xyz="0 0 1."/>
+        <parent link="world"/>
+        <child link="anchor"/>
     </joint>
   <link name="anchor">
@@ -63,6 +35,6 @@
     <inertial>
       <origin rpy="0 0 0" xyz="0 0 0.0"/>
-      <mass value="100.0"/>
-      <inertia ixx="10." ixy="0.0" ixz="0.0" iyy="10." iyz="0.0" izz="10."/>
+      <mass value="10.0"/>
+      <inertia ixx="0.1" ixy="0.0" ixz="0.0" iyy="0.1" iyz="0.0" izz="0.1"/>
     </inertial>
   </link>
@@ -70,5 +42,5 @@
   <joint name="mountain_wire_pitch" type="revolute">
     <parent link="anchor"/>
-    <child link="pre-wire1"/>
+    <child link="pre_wire1"/>
     <limit effort="1000" velocity="100.0" lower="-100" upper="100"/>
     <!-- joint rotates about y axis -->
@@ -78,5 +50,5 @@
     <dynamics damping="0.0" friction="0.0"/>
   </joint>
-  <link name="pre-wire1">
+  <link name="pre_wire1">
     <visual>
       <origin rpy="0 0 0" xyz="0 0 0"/>
@@ -102,6 +74,6 @@
   <!-- Revolute roll joint between the mountain and the wire -->
   <joint name="mountain_wire_roll" type="revolute">
-    <parent link="pre-wire1"/>
-    <child link="pre-wire2"/>
+    <parent link="pre_wire1"/>
+    <child link="pre_wire2"/>
     <limit effort="1000" velocity="100.0" lower="-100" upper="100"/>
     <!-- joint rotates about x axis -->
@@ -111,5 +83,5 @@
     <dynamics damping="0.0" friction="0.0"/>
   </joint>
-  <link name="pre-wire2">
+  <link name="pre_wire2">
     <visual>
       <origin rpy="0 0 0" xyz="0 0 0"/>
@@ -135,5 +107,5 @@
   <!-- Revolute yaw joint between the mountain and the wire -->
   <joint name="mountain_wire_yaw" type="revolute">
-    <parent link="pre-wire2"/>
+    <parent link="pre_wire2"/>
     <child link="wire"/>
     <limit effort="1000" velocity="100.0" lower="-100" upper="100"/>
@@ -147,6 +119,6 @@
     <inertial>
       <origin rpy="0 0 0" xyz="0 0 0.0"/>
-      <mass value="0.01"/>
-      <inertia ixx="0.0001" ixy="0.0" ixz="0.0" iyy="0.0001" iyz="0.0" izz="1e-6"/>
+      <mass value="0.5"/>
+      <inertia ixx="0.001" ixy="0.0" ixz="0.0" iyy="0.001" iyz="0.0" izz="0.001"/>
     </inertial>
   </link>
@@ -158,5 +130,5 @@
     <!-- joint translates on x axis -->
     <axis xyz="0 0 1"/>
-    <origin rpy="0 0 0" xyz="0.0 0.0 -1.0"/>
+    <origin rpy="0 0 0" xyz="0.0 0.0 0.0"/>
     <!-- pybullet simulation parameters -->
     <dynamics damping="0.0" friction="0.0"/>

Commit message: important! removing  mountain_wire_yaw joint that is redundant

File: urdf/climbingrobot.transmission.xacro (robot description, xacro)
@@ -18,14 +18,4 @@
                         </joint>
                         <actuator name="mountain_wire_roll">
-                                <hardwareInterface>hardware_interface/EffortJointInterface</hardwareInterface>
-                                <mechanicalReduction>1</mechanicalReduction>
-                        </actuator>
-                </transmission>
-		<transmission name="mountain_wire_yaw">
-                        <type>transmission_interface/SimpleTransmission</type>
-                        <joint name="mountain_wire_yaw">
-                                <hardwareInterface>hardware_interface/EffortJointInterface</hardwareInterface>
-                        </joint>
-                        <actuator name="mountain_wire_yaw">
                                 <hardwareInterface>hardware_interface/EffortJointInterface</hardwareInterface>
                                 <mechanicalReduction>1</mechanicalReduction>

File: urdf/climbingrobot.xacro (robot description, xacro)
@@ -65,41 +65,8 @@
   <joint name="mountain_wire_roll" type="revolute">
     <parent link="pre_wire1"/>
-    <child link="pre_wire2"/>
+    <child link="wire"/>
     <limit effort="1000" velocity="100.0" lower="-100" upper="100"/>
     <!-- joint rotates about x axis -->
     <axis xyz="1 0 0"/>
-    <origin rpy="0 0 0" xyz="0.0 0.0 0.0"/>
-    <!-- pybullet simulation parameters -->
-    <dynamics damping="0.0" friction="0.0"/>
-  </joint>
-  <link name="pre_wire2">
-    <visual>
-      <origin rpy="0 0 0" xyz="0 0 0"/>
-      <geometry>
-        <mesh filename="package://climbingrobot_description/meshes/obj/cylinder.obj" scale="0.01 0.01 0.01"/>
-      </geometry>
-      <material name="grey">
-        <color rgba=".7 .7 .7 .5"/>
-      </material>
-    </visual>
-    <collision>
-      <origin rpy="0 0 0" xyz="0 0 0.0"/>
-      <geometry>
-        <cylinder length="0.01" radius="0.01"/>
-      </geometry>
-    </collision>
-    <inertial>
-      <origin rpy="0 0 0" xyz="0 0 0.0"/>
-      <mass value="0.01"/>
-      <inertia ixx="0.0001" ixy="0.0" ixz="0.0" iyy="0.0001" iyz="0.0" izz="0.0001"/>
-    </inertial>
-  </link>
-  <!-- Revolute yaw joint between the mountain and the wire -->
-  <joint name="mountain_wire_yaw" type="revolute">
-    <parent link="pre_wire2"/>
-    <child link="wire"/>
-    <limit effort="1000" velocity="100.0" lower="-100" upper="100"/>
-    <!-- joint rotates about z axis -->
-    <axis xyz="0 0 1"/>
     <origin rpy="0 0 0" xyz="0.0 0.0 0.0"/>
     <!-- pybullet simulation parameters -->
