Commit message: added possibility to have a seond pillar, added anchor ball and target ball (commented)

File: urdf/climb_wall_2pillars.xacro (robot description, xacro)
@@ -6,10 +6,4 @@
  <material name="Red">
     <color rgba="${255/255} ${100/255} ${0/255} 1.0"/>
-  </material>
- <material name="Brown">
-    <color rgba="${198/255} ${94/255} ${42/255} 1.0"/>
-  </material>
- <material name="DarkBrown">
-    <color rgba="${144/255} ${68/255} ${30/255} 1.0"/>
   </material>
  <!--https://www.textures.com/browse/cliffs/2060 -->
@@ -30,5 +24,5 @@
 				<box size="0.1 $(arg anchorZ) $(arg anchorZ)"/>
 			</geometry>
-			<material name="Brown"/><!--rviz"/-->
+			<material name="Black"/><!--rviz"/-->
 		</visual>
 	        <collision name="box">
@@ -78,5 +72,5 @@
                           <mesh filename="package://climbingrobot_description/meshes/cone.stl" scale="1 1 1"/>
                         </geometry>
-			<material name="DarkBrown"/><!--rviz"/-->
+			<material name="Red"/><!--rviz"/-->
 		</visual>
 	        <collision>
@@ -88,4 +82,37 @@
 	       </collision>
 	</link>
+<!--
+	<gazebo reference="pillar2">
+   	 <material>Gazebo/RockWall</material>
+  	</gazebo> -->
+<!--
+	  <joint name="base_pillar2" type="fixed">
+	    <parent link="wall"/>
+	    <child link="pillar2"/>
+	    <origin rpy="0 0 0" xyz="0 0.0 0"/>
+	  </joint>-->
+<!--
+		<link name="pillar2">
+		<inertial>
+ 	        <mass value="10"/>
+ 	        <inertia ixx="0.4" ixy="0.0" ixz="0.0" iyy="0.4" iyz="0.0" izz="0.2"/>
+  	        </inertial>
+		<visual >
+			<!-- dont put name otherwise gazebo discards color-->
+<!-- 			<origin xyz="0  $(arg pillar2_posY) $(arg pillar2_posZ)"/>
+		        <geometry>
+                          <mesh filename="package://climbingrobot_description/meshes/cone.stl" scale="1 1 1"/>
+                        </geometry>
+			<material name="Red"/><!--rviz"/-->
+<!--
+		</visual>
+	        <collision>
+		       <origin xyz="0   $(arg pillar2_posY)  $(arg pillar2_posZ)"/>
+		  	 <origin xyz="0 0 0"/>
+		        <geometry>
+                          <mesh filename="package://climbingrobot_description/meshes/cone.stl" scale="1 1 1"/>
+                        </geometry>
+<!--	       </collision>
+	</link>-->
 	</xacro:if>
 	<gazebo>

File: urdf/climbingrobot.xacro (robot description, xacro)
@@ -17,8 +17,8 @@
         <child link="anchor"/>
     </joint>
-   <link name="anchor">
+    <link name="anchor">
     <visual>
 	<geometry>
-         <sphere radius="0.03" />
+         <sphere radius="0.4" />
 	</geometry>
     </visual>
@@ -29,4 +29,23 @@
     </inertial>
   </link>
+<!--
+    <joint name="target_link" type="fixed">
+        <origin rpy="0 0 0" xyz=" 3.   3. 0."/>
+        <parent link="world"/>
+        <child link="target"/>
+    </joint>-->
+<!--
+    <link name="target">
+    <visual>
+	<geometry>
+         <sphere radius="0.4" />
+	</geometry>
+    </visual>-->
+  <!--<inertial>
+      <origin rpy="0 0 0" xyz="0 0 0.0"/>
+      <mass value="0.01"/>
+      <inertia ixx="0.01" ixy="0.0" ixz="0.0" iyy="0.01" iyz="0.0" izz="0.01"/>
+    </inertial>
+  </link>-->
   <!-- Revolute pitch joint between the mountain and the wire -->
   <joint name="mountain_wire_pitch" type="revolute">
@@ -158,5 +177,5 @@
       <origin rpy="0 0 0" xyz="0 0 0"/>
       <geometry>
-        <mesh filename="package://climbingrobot_description/meshes/obj/with_foot/solo_body.obj" scale="1 1 1"/>
+        <mesh filename="package://climbingrobot_description/meshes/obj/with_foot/solo_body.obj" scale="2 2 2"/>
       </geometry>
       <material name="red">
