Commit message: setting higher effort limits and better masses

File: urdf/climbingrobot.xacro (robot description, xacro)
@@ -10,19 +10,19 @@
     </xacro:include>
     <xacro:include filename="$(find climbingrobot_description)/urdf/climbingrobot.transmission.xacro"/>
- 	<link name="world"/>
- 	<joint name="anchor_x_joint" type="prismatic">
-		<parent link="world"/>
-		<child link="fake_link1"/>
-		<axis xyz="1 0 0 "/>
-		<origin xyz="0 0 0" rpy="0 0 0"/>
-		<limit effort="1000" velocity="100.0" lower="-100" upper="100"/>
-	</joint>
-	<link name="fake_link1">
+    <link name="world"/>
+    <joint name="anchor_x_joint" type="prismatic">
+	<parent link="world"/>
+	<child link="fake_link1"/>
+	<axis xyz="1 0 0 "/>
+	<origin xyz="0 0 0" rpy="0 0 0"/>
+	<limit effort="1000" velocity="100.0" lower="-100" upper="100"/>
+    </joint>
+    <link name="fake_link1">
 	<inertial>
 	<mass value="0.00001"/>
 	<inertia ixx="5.8083e-4" ixy="0" ixz="0" iyy="3.0833e-5" iyz="0" izz="5.9083e-4"/>
 	</inertial>
-	</link>
-	<joint name="anchor_y_joint" type="prismatic">
+    </link>
+    <joint name="anchor_y_joint" type="prismatic">
 		<parent link="fake_link1"/>
 		<child link="fake_link2"/>
@@ -30,12 +30,12 @@
 		<origin xyz="0 0 0" rpy="0 0 0"/>
 		<limit effort="1000" velocity="100.0" lower="-100" upper="100"/>
-	</joint>
-	<link name="fake_link2">
+    </joint>
+    <link name="fake_link2">
 	<inertial>
 	<mass value="0.00001"/>
 	<inertia ixx="5.8083e-4" ixy="0" ixz="0" iyy="3.0833e-5" iyz="0" izz="5.9083e-4"/>
 	</inertial>
-	</link>
-	<joint name="anchor_z_joint" type="prismatic">
+    </link>
+    <joint name="anchor_z_joint" type="prismatic">
 		<parent link="fake_link2"/>
 		<child link="anchor"/>
@@ -43,5 +43,5 @@
 		<origin xyz="0 0 0" rpy="0 0 0"/>
 		<limit effort="1000" velocity="100.0" lower="-100" upper="100"/>
-	</joint>
+    </joint>
   <link name="anchor">
     <!--<visual>
@@ -63,6 +63,6 @@
     <inertial>
       <origin rpy="0 0 0" xyz="0 0 0.0"/>
-      <mass value="1.0"/>
-      <inertia ixx="1.0" ixy="0.0" ixz="0.0" iyy="1.0" iyz="0.0" izz="1.0"/>
+      <mass value="100.0"/>
+      <inertia ixx="10." ixy="0.0" ixz="0.0" iyy="10." iyz="0.0" izz="10."/>
     </inertial>
   </link>
@@ -71,5 +71,5 @@
     <parent link="anchor"/>
     <child link="pre-wire1"/>
-    <limit effort="3" lower="-10" upper="10" velocity="1000"/>
+    <limit effort="1000" velocity="100.0" lower="-100" upper="100"/>
     <!-- joint rotates about y axis -->
     <axis xyz="0 1 0"/>
@@ -104,5 +104,5 @@
     <parent link="pre-wire1"/>
     <child link="pre-wire2"/>
-    <limit effort="3" lower="-10" upper="10" velocity="1000"/>
+    <limit effort="1000" velocity="100.0" lower="-100" upper="100"/>
     <!-- joint rotates about x axis -->
     <axis xyz="1 0 0"/>
@@ -137,5 +137,5 @@
     <parent link="pre-wire2"/>
     <child link="wire"/>
-    <limit effort="3" lower="-10" upper="10" velocity="1000"/>
+    <limit effort="1000" velocity="100.0" lower="-100" upper="100"/>
     <!-- joint rotates about z axis -->
     <axis xyz="0 0 1"/>
@@ -155,5 +155,5 @@
     <parent link="wire"/>
     <child link="pre-base1"/>
-    <limit effort="3" lower="-10" upper="10" velocity="1000"/>
+    <limit effort="1000" velocity="100.0" lower="-100" upper="100"/>
     <!-- joint translates on x axis -->
     <axis xyz="0 0 1"/>
@@ -173,5 +173,5 @@
     <parent link="pre-base1"/>
     <child link="pre-base2"/>
-    <limit effort="3" lower="-10" upper="10" velocity="1000"/>
+    <limit effort="1000" velocity="100.0" lower="-100" upper="100"/>
     <!-- joint rotates about y axis -->
     <axis xyz="0 1 0"/>
@@ -191,5 +191,5 @@
     <parent link="pre-base2"/>
     <child link="pre-base3"/>
-    <limit effort="3" lower="-10" upper="10" velocity="1000"/>
+    <limit effort="1000" velocity="100.0" lower="-100" upper="100"/>
     <!-- joint rotates about x axis -->
     <axis xyz="1 0 0"/>
@@ -209,5 +209,5 @@
     <parent link="pre-base3"/>
     <child link="base_link"/>
-    <limit effort="3" lower="-10" upper="10" velocity="1000"/>
+    <limit effort="1000" velocity="100.0" lower="-100" upper="100"/>
     <!-- joint rotates about z axis -->
     <axis xyz="0 0 1"/>
@@ -223,5 +223,5 @@
       <mass value="1.0"/>
       <!-- The base is extremely symmetrical. -->
-      <inertia ixx="1.0" ixy="0.0" ixz="0.0" iyy="1.0" iyz="0.0" izz="1.0"/>
+      <inertia ixx="0.1" ixy="0.0" ixz="0.0" iyy="0.1" iyz="0.0" izz="0.1"/>
     </inertial>
     <!-- BASE LINK VISUAL -->
@@ -253,5 +253,5 @@
     <parent link="base_link"/>
     <child link="upper_link1"/>
-    <limit effort="3" lower="-10" upper="10" velocity="1000"/>
+    <limit effort="1000" velocity="100.0" lower="-100" upper="100"/>
     <!-- joints rotates around the y-axis -->
     <axis xyz="0 1 0"/>
@@ -296,5 +296,5 @@
     <parent link="upper_link1"/>
     <child link="upper_link2"/>
-    <limit effort="3" lower="-10" upper="10" velocity="1000"/>
+    <limit effort="1000" velocity="100.0" lower="-100" upper="100"/>
     <!-- joints rotates around the y-axis -->
     <axis xyz="1 0 0"/>
@@ -341,5 +341,5 @@
     <parent link="upper_link2"/>
     <child link="lower_link"/>
-    <limit effort="3" lower="-10" upper="10" velocity="1000"/>
+    <limit effort="1000" velocity="100.0" lower="-100" upper="100"/>
     <!-- joints rotates around the y-axis -->
     <axis xyz="0 0 1"/>

Commit message: passing anchorZ as param, adding wall (does not compute contacts)

File: urdf/climbingrobot.xacro (robot description, xacro)
@@ -5,4 +5,5 @@
     <xacro:arg name="robot_name" default="climbingrobot"/>
     <xacro:arg name="new_gazebo_version" default="false"/>
+    <xacro:arg name="anchorZ" default="5."/>
     <xacro:include filename="$(find climbingrobot_description)/gazebo/gazebo.urdf.xacro">
         <xacro:arg name="task_period" value="$(arg task_period)"/>
@@ -12,25 +13,24 @@
     <link name="world"/>
    <joint name="mountain" type="fixed">
-        <origin rpy="0 0 0" xyz="0 0 1."/>
+        <origin rpy="0 0 0" xyz="0 0 $(arg anchorZ)"/>
         <parent link="world"/>
         <child link="anchor"/>
     </joint>
   <link name="anchor">
-    <!--<visual>
-      <origin rpy="0 0 0" xyz="0 0 0"/>
-      <geometry>
-        <mesh filename="package://climbingrobot_description/meshes/obj/cube.obj" scale="0.01 10.0 10.0"/>
+    <visual>
+      <origin rpy="0. -0.1 0" xyz="-0.25 0 ${-$(arg anchorZ)/2.0}"/>
+      <geometry>
+         <box size="0.1 $(arg anchorZ) $(arg anchorZ)"/>
       </geometry>
       <material name="ground">
-        <color rgba=".9 .1 .1 .5"/>
-      </material>
-    </visual>-->
-    <!-- TODO manage wall collision-->
-    <!--collision>
-      <origin rpy="0 0 0" xyz="0 0 0.0"/>
-      <geometry>
-        <box size="0.1 10.0 10.0"/>
-      </geometry>
-    </collision-->
+        <color rgba="0. 1 0"/>
+      </material>
+    </visual>
+    <collision>
+      <origin rpy="0 -0.1 0" xyz="-0.25 0  ${-$(arg anchorZ)/2.0}"/>
+      <geometry>
+        <box size="0.1 $(arg anchorZ) $(arg anchorZ)"/>
+      </geometry>
+    </collision>
     <inertial>
       <origin rpy="0 0 0" xyz="0 0 0.0"/>
@@ -376,5 +376,5 @@
       <origin rpy="0 0 0" xyz="0 0 0"/>
       <geometry>
-        <mesh filename="package://climbingrobot_description/meshes/obj/with_foot/solo_foot.obj"/>
+        <sphere radius="0.02175" />
       </geometry>
 	<material name="black">
@@ -386,5 +386,5 @@
       <origin rpy="0 0 0" xyz="0 0 0"/>
       <geometry>
-        <mesh filename="package://climbingrobot_description/meshes/obj/with_foot/solo_foot.obj"/>
+        <sphere radius="0.02175" />
       </geometry>
       <material name="grey">
@@ -392,9 +392,4 @@
       </material>
     </collision>
-    <!-- Bullet specific paramters -->
-    <contact>
-      <lateral_friction value="1.0"/>
-      <restitution value="0.5"/>
-    </contact>
   </link>
   <!-- END LOWER LEG LINK -->

Commit message: removed wall because it was not computing contacts

File: urdf/climbingrobot.xacro (robot description, xacro)
@@ -19,18 +19,8 @@
   <link name="anchor">
     <visual>
-      <origin rpy="0. -0.1 0" xyz="-0.25 0 ${-$(arg anchorZ)/2.0}"/>
-      <geometry>
-         <box size="0.1 $(arg anchorZ) $(arg anchorZ)"/>
-      </geometry>
-      <material name="ground">
-        <color rgba="0. 1 0"/>
-      </material>
-    </visual>
-    <collision>
-      <origin rpy="0 -0.1 0" xyz="-0.25 0  ${-$(arg anchorZ)/2.0}"/>
-      <geometry>
-        <box size="0.1 $(arg anchorZ) $(arg anchorZ)"/>
-      </geometry>
-    </collision>
+	<geometry>
+         <sphere radius="0.03" />
+	</geometry>
+    </visual>
     <inertial>
       <origin rpy="0 0 0" xyz="0 0 0.0"/>

Commit message: changes to be consistent with theta phi l definitions

File: urdf/climbingrobot.xacro (robot description, xacro)
@@ -5,5 +5,5 @@
     <xacro:arg name="robot_name" default="climbingrobot"/>
     <xacro:arg name="new_gazebo_version" default="false"/>
-    <xacro:arg name="anchorZ" default="5."/>
+    <xacro:arg name="anchorZ" default="1."/>
     <xacro:include filename="$(find climbingrobot_description)/gazebo/gazebo.urdf.xacro">
         <xacro:arg name="task_period" value="$(arg task_period)"/>
@@ -35,5 +35,5 @@
     <limit effort="1000" velocity="100.0" lower="-100" upper="100"/>
     <!-- joint rotates about y axis -->
-    <axis xyz="0 1 0"/>
+    <axis xyz="0 -1 0"/>
     <origin rpy="0 0 0" xyz="0.0 0.0 0.0"/>
     <!-- pybullet simulation parameters -->
@@ -119,5 +119,5 @@
     <limit effort="1000" velocity="100.0" lower="-100" upper="100"/>
     <!-- joint translates on x axis -->
-    <axis xyz="0 0 1"/>
+    <axis xyz="0 0 -1"/>
     <origin rpy="0 0 0" xyz="0.0 0.0 0.0"/>
     <!-- pybullet simulation parameters -->

Commit message: changing definition of hip pitch and hip roll joints
increasing base link mass to 5 kg

File: urdf/climbingrobot.xacro (robot description, xacro)
@@ -183,5 +183,5 @@
       <origin rpy="0 0 0" xyz="0 0 0"/>
       <!-- <mass value="0.36"/> -->
-      <mass value="1.0"/>
+      <mass value="5.0"/>
       <!-- The base is extremely symmetrical. -->
       <inertia ixx="0.1" ixy="0.0" ixz="0.0" iyy="0.1" iyz="0.0" izz="0.1"/>
@@ -217,5 +217,5 @@
     <limit effort="1000" velocity="100.0" lower="-100" upper="100"/>
     <!-- joints rotates around the y-axis -->
-    <axis xyz="0 1 0"/>
+    <axis xyz="0 -1 0"/>
     <origin rpy="0 0 0" xyz="0.0 -0.02 0.025"/>
     <!-- pybullet simulation parameters -->
@@ -260,5 +260,5 @@
     <limit effort="1000" velocity="100.0" lower="-100" upper="100"/>
     <!-- joints rotates around the y-axis -->
-    <axis xyz="1 0 0"/>
+    <axis xyz="-1 0 0"/>
     <origin rpy="0 0 0" xyz="0.0 0.0 0.0"/>
     <!-- pybullet simulation parameters -->

Commit message: fixing inertias and masses
total robot mass 6.5 kg

File: urdf/climbingrobot.xacro (robot description, xacro)
@@ -17,5 +17,5 @@
         <child link="anchor"/>
     </joint>
-  <link name="anchor">
+   <link name="anchor">
     <visual>
 	<geometry>
@@ -25,6 +25,6 @@
     <inertial>
       <origin rpy="0 0 0" xyz="0 0 0.0"/>
-      <mass value="10.0"/>
-      <inertia ixx="0.1" ixy="0.0" ixz="0.0" iyy="0.1" iyz="0.0" izz="0.1"/>
+      <mass value="0.01"/>
+      <inertia ixx="0.01" ixy="0.0" ixz="0.0" iyy="0.01" iyz="0.0" izz="0.01"/>
     </inertial>
   </link>
@@ -109,5 +109,5 @@
     <inertial>
       <origin rpy="0 0 0" xyz="0 0 0.0"/>
-      <mass value="0.5"/>
+      <mass value="0.01"/>
       <inertia ixx="0.001" ixy="0.0" ixz="0.0" iyy="0.001" iyz="0.0" izz="0.001"/>
     </inertial>
@@ -185,5 +185,5 @@
       <mass value="5.0"/>
       <!-- The base is extremely symmetrical. -->
-      <inertia ixx="0.1" ixy="0.0" ixz="0.0" iyy="0.1" iyz="0.0" izz="0.1"/>
+      <inertia ixx="0.5" ixy="0.0" ixz="0.0" iyy="0.5" iyz="0.0" izz="0.5"/>
     </inertial>
     <!-- BASE LINK VISUAL -->
@@ -226,6 +226,6 @@
     <inertial>
       <origin rpy="0 0 0" xyz="0.0000 0.0 -0.0"/>
-      <mass value="0.01"/>
-      <inertia ixx="0.00041107" ixy="0.0" ixz="0.0" iyy="0.00041193" iyz="0.00004671" izz="0.00003024"/>
+      <mass value="0.5"/>
+      <inertia ixx="0.01" ixy="0.0" ixz="0.0" iyy="0.01" iyz="0.00004671" izz="0.01"/>
     </inertial>
     <!-- UPPER LEG LINK VISUAL
@@ -269,6 +269,6 @@
     <inertial>
       <origin rpy="0 0 0" xyz="0.0000 0.0 -0.0"/>
-      <mass value="0.14853845"/>
-      <inertia ixx="0.00041107" ixy="0.0" ixz="0.0" iyy="0.00041193" iyz="0.00004671" izz="0.00003024"/>
+      <mass value="0.5"/>
+      <inertia ixx="0.01" ixy="0.0" ixz="0.0" iyy="0.01" iyz="0.00004671" izz="0.01"/>
     </inertial>
     <!-- UPPER LEG LINK VISUAL -->
@@ -314,6 +314,6 @@
     <inertial>
       <origin rpy="0 0 0" xyz="0.0 0.0 -0.09"/>
-      <mass value="0.0307"/>
-      <inertia ixx="0.00012024" ixy="0.0" ixz="0.0" iyy="0.00012029" iyz="0.00000305" izz="0.00000216"/>
+      <mass value="0.5"/>
+      <inertia ixx="0.01" ixy="0.0" ixz="0.0" iyy="0.01" iyz="0.00000305" izz="0.01"/>
     </inertial>
     <!-- LOWER LEG LINK VISUAL -->

Commit message: adding foot sensor

File: urdf/climbingrobot.xacro (robot description, xacro)
@@ -352,4 +352,27 @@
   <!-- END LOWER LEG LINK -->
   <!-- Joint between the base and the ${prefix} upper leg -->
+    <gazebo reference="foot">
+        <kp>1000000.0</kp>
+        <kd>100.0</kd>
+        <mu1>0.8</mu1>
+        <mu2>0.8</mu2>
+        <maxVel>1.0</maxVel>
+        <maxContacts>1</maxContacts>
+        <sensor name="foot_contact_sensor" type="contact">
+                <always_on>true</always_on>
+                <update_rate>1000.0</update_rate>
+                <contact>
+                <collision>lower_link_fixed_joint_lump__foot_collision_1</collision>
+                </contact>
+                <!-- the sensor readings in terms of force torques are expressed in the lowerleg frame
+                because gazebo lumps the fake footframe with the real parent link, the normals are in the world frame-->
+                <plugin name="foot_bumper" filename="libgazebo_ros_bumper.so">
+                        <bumperTopicName>/$(arg robot_name)/foot_bumper</bumperTopicName>
+                        <!--robotNamespace>solo</robotNamespace-->
+                        <frameName>foot</frameName>
+                </plugin>
+        </sensor>
+        <material>Gazebo/Black</material>
+   </gazebo>
    <xacro:climbingrobot_transmission/>
 </robot>

Commit message: added rope  drawing to gazebo

File: urdf/climbingrobot.xacro (robot description, xacro)
@@ -111,4 +111,22 @@
   </joint>
   <link name="pre-base1">
+      <visual>
+      <origin rpy="0 0 0" xyz="0 0 ${$(arg anchorZ)/2}"/>
+      <geometry>
+        <cylinder radius="0.05" length="$(arg anchorZ)"/>
+      </geometry>
+      <material name="grey">
+        <color rgba=".7 .7 .7 .5"/>
+      </material>
+    </visual>
+   <collision>
+      <origin rpy="0 0 0" xyz="0 0 ${$(arg anchorZ)/2}"/>
+      <geometry>
+        <cylinder radius="0.05" length="$(arg anchorZ)"/>
+      </geometry>
+      <material name="grey">
+        <color rgba=".7 .7 .7 .5"/>
+      </material>
+    </collision>
     <inertial>
       <origin rpy="0 0 0" xyz="0 0 0.0"/>

Commit message: reverting scale changed for mistake

File: urdf/climbingrobot.xacro (robot description, xacro)
@@ -195,5 +195,5 @@
       <origin rpy="0 0 0" xyz="0 0 0"/>
       <geometry>
-        <mesh filename="package://climbingrobot_description/meshes/obj/with_foot/solo_body.obj" scale="2 2 2"/>
+        <mesh filename="package://climbingrobot_description/meshes/obj/with_foot/solo_body.obj" scale="1 1 1"/>
       </geometry>
       <material name="red">
