Commit message: added wheels with bumpers

File: urdf/climbingrobot2landing.transmission.xacro (robot description, xacro)
@@ -172,4 +172,24 @@
                         </actuator>
                 </transmission>
+      		<transmission name="wheel_joint_l">
+                        <type>transmission_interface/SimpleTransmission</type>
+                        <joint name="wheel_joint_l">
+                                <hardwareInterface>hardware_interface/EffortJointInterface</hardwareInterface>
+                        </joint>
+                        <actuator name="wheel_joint_l">
+                                <hardwareInterface>hardware_interface/EffortJointInterface</hardwareInterface>
+                                <mechanicalReduction>1</mechanicalReduction>
+                        </actuator>
+                </transmission>
+   	        <transmission name="wheel_joint_r">
+                        <type>transmission_interface/SimpleTransmission</type>
+                        <joint name="wheel_joint_r">
+                                <hardwareInterface>hardware_interface/EffortJointInterface</hardwareInterface>
+                        </joint>
+                        <actuator name="wheel_joint_r">
+                                <hardwareInterface>hardware_interface/EffortJointInterface</hardwareInterface>
+                                <mechanicalReduction>1</mechanicalReduction>
+                        </actuator>
+                </transmission>
         </xacro:macro>
 </robot>

File: urdf/climbingrobot2landing.xacro (robot description, xacro)
@@ -13,5 +13,6 @@
    <xacro:arg name="hoist_distance" default="0.1"/>
    <xacro:arg name="hoist_base_distanceZ" default="0.05"/>
-   <xacro:arg name="lowerleg_landing_length" default="0.4"/>
+   <xacro:arg name="lowerleg_landing_length" default="0.3"/>
+    <xacro:property name="WHEEL_pos" value="0.10183" />
     <xacro:include filename="$(find climbingrobot_description)/gazebo/gazebo.urdf.xacro">
         <xacro:arg name="task_period" value="$(arg task_period)"/>
@@ -401,5 +402,5 @@
     <!-- joints rotates around the z-axis -->
     <axis xyz="0 0 1"/>
-    <origin rpy="0 0 1.57" xyz="0.0 -0.08 -0.05"/>
+    <origin rpy="0 0 1.57" xyz="0.0 -0.08 0.025"/>
     <!-- pybullet simulation parameters -->
     <dynamics damping="0.0" friction="0.0"/>
@@ -460,5 +461,5 @@
     </collision>
    </link>
- <gazebo reference="foot_landing_l">
+ <gazebo reference="wheel_l">
         <kp>1000000.0</kp>
         <kd>100.0</kd>
@@ -471,5 +472,5 @@
                 <update_rate>1000.0</update_rate>
                 <contact>
-                <collision>lowerleg_landing_l_fixed_joint_lump__foot_landing_l_collision</collision>
+                <collision>wheel_l_collision</collision>
                 </contact>
                 <!-- the sensor readings in terms of force torques are expressed in the lowerleg frame
@@ -478,5 +479,5 @@
                         <bumperTopicName>/$(arg robot_name)/foot_landing_l_bumper</bumperTopicName>
                         <!--robotNamespace>solo</robotNamespace-->
-                        <frameName>foot_landing_l</frameName>
+                        <frameName>wheel_l</frameName>
                 </plugin>
         </sensor>
@@ -490,5 +491,5 @@
     <!-- joints rotates around the z-axis -->
     <axis xyz="0 0 1"/>
-    <origin rpy="0 0 -1.57" xyz="0.0 0.08 -0.05"/>
+    <origin rpy="0 0 -1.57" xyz="0.0 0.08 0.025"/>
     <!-- pybullet simulation parameters -->
     <dynamics damping="0.0" friction="0.0"/>
@@ -549,5 +550,5 @@
     </collision>
    </link>
-    <gazebo reference="foot_landing_r">
+    <gazebo reference="wheel_r">
         <kp>1000000.0</kp>
         <kd>100.0</kd>
@@ -560,5 +561,5 @@
                 <update_rate>1000.0</update_rate>
                 <contact>
-                <collision>lowerleg_landing_r_fixed_joint_lump__foot_landing_r_collision</collision>
+                <collision>wheel_r_collision</collision>
                 </contact>
                 <!-- the sensor readings in terms of force torques are expressed in the lowerleg frame
@@ -567,9 +568,76 @@
                         <bumperTopicName>/$(arg robot_name)/foot_landing_r_bumper</bumperTopicName>
                         <!--robotNamespace>solo</robotNamespace-->
-                        <frameName>foot_landing_r</frameName>
+                        <frameName>wheel_r</frameName>
                 </plugin>
         </sensor>
         <material>Gazebo/Black</material>
    </gazebo>
+    <!--WHEEL JOINTS-->
+        <joint name="wheel_joint_l" type="revolute">
+            <parent link="foot_landing_l"/>
+            <child link="wheel_l"/>
+            <axis xyz="1 0 0"/>
+            <origin xyz="-${WHEEL_pos} 0  0" rpy="0 -1.57 0" />
+            <limit effort="100" lower="-1e10" upper="1e10" velocity="100"/>
+            <dynamics damping="0.0" friction="0.0"/>
+        </joint>
+        <!-- WHEEL ASSEMBLY -->
+        <link name="wheel_l">
+            <!--VISUAL-->
+            <visual>
+                <origin xyz="0 0 0" rpy="0 0 0" />
+                <geometry>
+                       <mesh filename="package://climbingrobot_description/meshes/wheel_y.stl"/>
+                </geometry>
+                       <material name="blue">
+       			 <color rgba="0 0 1  1.0"/>
+      		</material>
+            </visual>
+            <!--COLLISION-->
+            <collision>
+                <origin xyz="0 0 0" rpy="0 0 0" />
+                <geometry>
+                       <mesh filename="package://climbingrobot_description/meshes/wheel_y.stl"/>
+                </geometry>
+            </collision>
+               <inertial>
+                    <origin xyz="0 0 0" rpy="0 0 0"/>
+                    <mass value="0.00693606"/>
+                    <inertia ixx="0.00000057" ixy="0.0" ixz="0.0" iyy="0.00000084" iyz="0.0" izz="0.00000053"/>
+                </inertial>
+        </link>
+        <joint name="wheel_joint_r" type="revolute">
+            <parent link="foot_landing_r"/>
+            <child link="wheel_r"/>
+            <axis xyz="1 0 0"/>
+            <origin xyz="-${WHEEL_pos} 0  0" rpy="0 -1.57 0" />
+            <limit effort="100" lower="-1e10" upper="1e10" velocity="100"/>
+            <dynamics damping="0.0" friction="0.0"/>
+        </joint>
+        <!-- WHEEL ASSEMBLY -->
+        <link name="wheel_r">
+            <!--VISUAL-->
+            <visual>
+                <origin xyz="0 0 0" rpy="0 0 0" />
+                <geometry>
+                       <mesh filename="package://climbingrobot_description/meshes/wheel_y.stl"/>
+                </geometry>
+                  <material name="blue">
+       			 <color rgba="0 0 1  1.0"/>
+      		</material>
+            </visual>
+            <!--COLLISION-->
+            <collision>
+                <origin xyz="0 0 0" rpy="0 0 0" />
+                <geometry>
+                       <mesh filename="package://climbingrobot_description/meshes/wheel_y.stl"/>
+                </geometry>
+            </collision>
+               <inertial>
+                    <origin xyz="0 0 0" rpy="0 0 0"/>
+                    <mass value="0.00693606"/>
+                    <inertia ixx="0.00000057" ixy="0.0" ixz="0.0" iyy="0.00000084" iyz="0.0" izz="0.00000053"/>
+                </inertial>
+        </link>
   <!-- Joint between the base and the ${prefix} upper leg -->
   <joint name="hip_pitch" type="revolute">
