Commit message: adding mountain to visualization, in rviz
added color black to mountain

File: urdf/climb_wall.xacro (robot description, xacro)
@@ -1,5 +1,8 @@
 <?xml version="1.0" encoding="utf-8"?>
 <robot name="climb_wall" xmlns:xacro="http://ros.org/wiki/xacro">
-   <xacro:arg name="anchorZ" default="1."/>
+ <material name="Black">
+    <color rgba="${0/255} ${0/255} ${0/255} 1.0"/>
+  </material>
+<xacro:arg name="anchorZ" default="1."/>
 	<link name="wall">
 		<inertial>
@@ -7,6 +10,7 @@
  	        <inertia ixx="0.4" ixy="0.0" ixz="0.0" iyy="0.4" iyz="0.0" izz="0.2"/>
   	     </inertial>
-		<visual name="box">
+		<visual > <!-- dont put name otherwise gazebo discards color-->
  			<origin xyz="0 0 ${$(arg anchorZ)/2}"/>
+			<material name="Black"/> <!-- rviz will use this color -->
 			<geometry>
 				<box size="0.1 $(arg anchorZ) $(arg anchorZ)"/>

Commit message: adding some materials (not working yet)

File: urdf/climb_wall.xacro (robot description, xacro)
@@ -4,4 +4,5 @@
     <color rgba="${0/255} ${0/255} ${0/255} 1.0"/>
   </material>
+ <!--https://www.textures.com/browse/cliffs/2060 -->
 <xacro:arg name="anchorZ" default="1."/>
 	<link name="wall">
@@ -12,8 +13,8 @@
 		<visual > <!-- dont put name otherwise gazebo discards color-->
  			<origin xyz="0 0 ${$(arg anchorZ)/2}"/>
-			<material name="Black"/> <!-- rviz will use this color -->
 			<geometry>
 				<box size="0.1 $(arg anchorZ) $(arg anchorZ)"/>
 			</geometry>
+			<material name="Black"/><!--rviz"/-->
 		</visual>
 	        <collision name="box">
@@ -22,24 +23,4 @@
  				<box size="0.1 $(arg anchorZ) $(arg anchorZ)"/>
 	        	</geometry>
-			 <surface>
-			  <bounce>
-			    <restitution_coefficient>0.01</restitution_coefficient>
-			    <threshold>5.0</threshold>
-			  </bounce>
-			  <friction>
-			    <ode>
-			      <mu>1</mu>
-			      <mu2>1</mu2>
-			    </ode>
-			  </friction>
-			  <contact>
-			     <ode>
-				<max_vel>0.1</max_vel>
-				<min_depth>0.001</min_depth>
-				<kp>1000000.0</kp>
-				<kd>1000.0</kd>
-			      </ode>
-			    </contact>
-			</surface>
 	       </collision>
 	</link>
@@ -47,3 +28,7 @@
 	    <static>true</static>
 	</gazebo>
+	 <!--one of this /usr/share/gazebo-11/media/materials/scripts/gazebo.material   is for gazebo -->
+	<gazebo reference="wall">
+   	 <material>Gazebo/RockWall</material>
+  	</gazebo>
 </robot>

Commit message: added pillar obstacle

File: urdf/climb_wall.xacro (robot description, xacro)
@@ -4,6 +4,10 @@
     <color rgba="${0/255} ${0/255} ${0/255} 1.0"/>
   </material>
+ <material name="Red">
+    <color rgba="${255/255} ${0/255} ${0/255} 1.0"/>
+  </material>
  <!--https://www.textures.com/browse/cliffs/2060 -->
-<xacro:arg name="anchorZ" default="1."/>
+<xacro:arg name="obstacle" default="true"/>
+<xacro:arg name="anchorZ" default="10."/>
 	<link name="wall">
 		<inertial>
@@ -45,4 +49,34 @@
 	       </collision>
 	</link>
+	<xacro:if value="$(arg obstacle)">
+	<gazebo reference="pillar">
+   	 <material>Gazebo/RockWall</material>
+  	</gazebo>
+	  <joint name="base" type="fixed">
+	    <parent link="wall"/>
+	    <child link="pillar"/>
+	    <origin rpy="0 0 0" xyz="0 0.0 0"/>
+	  </joint>
+		<link name="pillar">
+		<inertial>
+ 	        <mass value="10"/>
+ 	        <inertia ixx="0.4" ixy="0.0" ixz="0.0" iyy="0.4" iyz="0.0" izz="0.2"/>
+  	        </inertial>
+		<visual > <!-- dont put name otherwise gazebo discards color-->
+ 			<origin xyz="0 2 0"/>
+		        <geometry>
+                          <mesh filename="package://climbingrobot_description/meshes/cone.stl" scale="1 1 1"/>
+                        </geometry>
+			<material name="Red"/><!--rviz"/-->
+		</visual>
+	        <collision>
+		       <origin xyz="0 2 0"/>
+		  	 <origin xyz="0 0 0"/>
+		        <geometry>
+                          <mesh filename="package://climbingrobot_description/meshes/cone.stl" scale="1 1 1"/>
+                        </geometry>
+	       </collision>
+	</link>
+	</xacro:if>
 	<gazebo>
 	    <static>true</static>

File: urdf/climbingrobot.xacro (robot description, xacro)
@@ -34,5 +34,5 @@
     <child link="pre_wire1"/>
     <limit effort="1000" velocity="100.0" lower="-100" upper="100"/>
-    <!-- joint rotates about y axis -->
+    <!-- joint rotates about -y axis -->
     <axis xyz="0 -1 0"/>
     <origin rpy="0 0 0" xyz="0.0 0.0 0.0"/>

Commit message: parametrized obstacle (default Y = 1.5)

File: urdf/climb_wall.xacro (robot description, xacro)
@@ -5,9 +5,11 @@
   </material>
  <material name="Red">
-    <color rgba="${255/255} ${0/255} ${0/255} 1.0"/>
+    <color rgba="${255/255} ${100/255} ${0/255} 1.0"/>
   </material>
  <!--https://www.textures.com/browse/cliffs/2060 -->
 <xacro:arg name="obstacle" default="true"/>
 <xacro:arg name="anchorZ" default="10."/>
+<xacro:arg name="pillar_posX" default="0"/>
+<xacro:arg name="pillar_posY" default="1.5"/>
 	<link name="wall">
 		<inertial>
@@ -64,5 +66,5 @@
   	        </inertial>
 		<visual > <!-- dont put name otherwise gazebo discards color-->
- 			<origin xyz="0 2 0"/>
+ 			<origin xyz="0  $(arg pillar_posY) 0"/>
 		        <geometry>
                           <mesh filename="package://climbingrobot_description/meshes/cone.stl" scale="1 1 1"/>
@@ -71,5 +73,5 @@
 		</visual>
 	        <collision>
-		       <origin xyz="0 2 0"/>
+		       <origin xyz="0   $(arg pillar_posY) 0"/>
 		  	 <origin xyz="0 0 0"/>
 		        <geometry>

Commit message: add wall_inclination parameter to climbingrobot2landing
removed base_link / upperleg collision for climbingrobot2landing to
avoid issues with leg retraction

File: urdf/climb_wall.xacro (robot description, xacro)
@@ -16,4 +16,5 @@
 <xacro:arg name="obstacle" default="true"/>
 <xacro:arg name="anchorZ" default="10."/>
+<xacro:arg name="wall_inclination" default="0.0"/>
 <xacro:arg name="pillar_posY" default="1.5"/>
 <xacro:arg name="pillar_posZ" default="0"/>
@@ -26,5 +27,5 @@
   	     </inertial>
 		<visual > <!-- dont put name otherwise gazebo discards color-->
- 			<origin xyz="0 0 ${$(arg anchorZ)/2}"/>
+ 			<origin xyz="${$(arg anchorZ)/2 *sin($(arg wall_inclination))}  0 ${$(arg anchorZ)/2}" rpy="0  -$(arg wall_inclination) 0"/>
 			<geometry>
 				<box size="0.1 $(arg anchorZ) $(arg anchorZ)"/>
@@ -33,5 +34,5 @@
 		</visual>
 	        <collision name="box">
-		       <origin xyz="0 0 ${$(arg anchorZ)/2}"/>
+		       <origin xyz="${$(arg anchorZ)/2 *sin($(arg wall_inclination))} 0 ${$(arg anchorZ)/2}" rpy="0  -$(arg wall_inclination) 0"/>
 		       <geometry>
  				<box size="0.1 $(arg anchorZ) $(arg anchorZ)"/>

File: urdf/climbingrobot2landing.xacro (robot description, xacro)
@@ -711,6 +711,6 @@
       </material>
     </visual>
-    <!-- UPPER LEG LINK COLLISION -->
-    <collision>
+    <!-- UPPER LEG LINK COLLISION  Commented to allow complete retraction without creating forces-->
+    <!--collision>
       <origin rpy="0 0 0" xyz="0 0 0"/>
       <geometry>
@@ -720,5 +720,5 @@
         	<color rgba="0.898 0.913 0.941 1.0"/>
     	</material>
-    </collision>
+    </collision-->
     <!-- Bullet specific paramters -->
     <contact>
@@ -756,5 +756,5 @@
     	</material>
     </visual>
-    <!-- LOWER LEG LINK COLLISION -->
+    <!-- LOWER LEG LINK COLLISION-->
     <collision>
       <origin rpy="0 0 0" xyz="0 0 0"/>
