Commit message: tuned obstacle  position for climbwall2

File: urdf/climb_wall2.xacro (robot description, xacro)
@@ -13,9 +13,12 @@
     <color rgba="${144/255} ${68/255} ${30/255} 1.0"/>
   </material>
+<material name="orange">
+  <color rgba="0.8 0.4 0.0 1.0"/>
+</material>
  <!--https://www.textures.com/browse/cliffs/2060 -->
 <xacro:arg name="obstacle" default="true"/>
 <xacro:arg name="anchorZ" default="10."/>
 <xacro:arg name="wall_inclination" default="0.0"/>
-<xacro:arg name="pillar_posX" default="0"/>
+<xacro:arg name="pillar_posX" default="-0.5"/>
 <xacro:arg name="pillar_posY" default="3"/>
 <xacro:arg name="pillar_posZ" default="-7.5"/>
@@ -60,7 +63,4 @@
 	</link>
 	<xacro:if value="$(arg obstacle)">
-		<gazebo reference="pillar">
-	   	 <material>Gazebo/RockWall</material>
-	  	</gazebo>
 		  <joint name="base_pillar" type="fixed">
 		    <parent link="wall"/>
@@ -68,22 +68,22 @@
 		    <origin rpy="0 0 0" xyz="0 0 0"/>
 		  </joint>
-			<link name="pillar">
-			<inertial>
-	 	        <mass value="10"/>
-	 	        <inertia ixx="0.4" ixy="0.0" ixz="0.0" iyy="0.4" iyz="0.0" izz="0.2"/>
-	  	        </inertial>
-			<visual > <!-- dont put name otherwise gazebo discards color-->
-	 			  <origin rpy="0 0 0" xyz="$(arg pillar_posX) $(arg pillar_posY)  ${$(arg anchorZ) + $(arg pillar_posZ)} "/>
-				<geometry>
-		                  <mesh filename="package://climbingrobot_description/meshes/ellipsoid.stl" scale="1 1 1"/>
-		                </geometry>
-				<material name="DarkBrown"/><!--rviz"/-->
-			</visual>
-			<collision>
- 				<origin rpy="0 0 0" xyz="$(arg pillar_posX) $(arg pillar_posY)  ${$(arg anchorZ) + $(arg pillar_posZ)} "/>
-				 <geometry>
-		                  <mesh filename="package://climbingrobot_description/meshes/ellipsoid.stl" scale="1 1 1"/>
-		                </geometry>
-		       </collision>
+		<link name="pillar">
+		<inertial>
+ 	        <mass value="10"/>
+ 	        <inertia ixx="0.4" ixy="0.0" ixz="0.0" iyy="0.4" iyz="0.0" izz="0.2"/>
+  	        </inertial>
+		<visual > <!-- dont put name otherwise gazebo discards color-->
+ 			  <origin rpy="0 0 0" xyz="$(arg pillar_posX) $(arg pillar_posY)  ${$(arg anchorZ) + $(arg pillar_posZ)} "/>
+			<geometry>
+	                  <mesh filename="package://climbingrobot_description/meshes/ellipsoid.stl" scale="1 1 1"/>
+	                </geometry>
+			 <material name="orange"/>
+		</visual>
+		<collision>
+			<origin rpy="0 0 0" xyz="$(arg pillar_posX) $(arg pillar_posY)  ${$(arg anchorZ) + $(arg pillar_posZ)} "/>
+			 <geometry>
+	                  <mesh filename="package://climbingrobot_description/meshes/ellipsoid.stl" scale="1 1 1"/>
+	                </geometry>
+	       </collision>
 		</link>
 	</xacro:if>
@@ -95,3 +95,6 @@
    	 <material>Gazebo/RockWall</material>
   	</gazebo>
+	<gazebo reference="pillar">
+   	 <material>Gazebo/RockWall</material>
+  	</gazebo>
 </robot>

Commit message: parametrized obstacle location

File: urdf/climb_wall2.xacro (robot description, xacro)
@@ -20,7 +20,7 @@
 <xacro:arg name="anchorZ" default="10."/>
 <xacro:arg name="wall_inclination" default="0.0"/>
-<xacro:arg name="pillar_posX" default="-0.5"/>
-<xacro:arg name="pillar_posY" default="3"/>
-<xacro:arg name="pillar_posZ" default="-7.5"/>
+<xacro:arg name="obstacle_x" default="-0.5"/>
+<xacro:arg name="obstacle_y" default="2.5"/>
+<xacro:arg name="obstacle_z" default="-6"/>
 	<link name="wall">
 		<inertial>
@@ -74,5 +74,5 @@
   	        </inertial>
 		<visual > <!-- dont put name otherwise gazebo discards color-->
- 			  <origin rpy="0 0 0" xyz="$(arg pillar_posX) $(arg pillar_posY)  ${$(arg anchorZ) + $(arg pillar_posZ)} "/>
+ 			  <origin rpy="0 0 0" xyz="$(arg obstacle_x) $(arg obstacle_y)  ${$(arg anchorZ) + $(arg obstacle_z)} "/>
 			<geometry>
 	                  <mesh filename="package://climbingrobot_description/meshes/ellipsoid.stl" scale="1 1 1"/>
@@ -81,5 +81,5 @@
 		</visual>
 		<collision>
-			<origin rpy="0 0 0" xyz="$(arg pillar_posX) $(arg pillar_posY)  ${$(arg anchorZ) + $(arg pillar_posZ)} "/>
+			<origin rpy="0 0 0" xyz="$(arg obstacle_x) $(arg obstacle_y)  ${$(arg anchorZ) + $(arg obstacle_z)} "/>
 			 <geometry>
 	                  <mesh filename="package://climbingrobot_description/meshes/ellipsoid.stl" scale="1 1 1"/>

Commit message: added obstacle_size

File: urdf/climb_wall2.xacro (robot description, xacro)
@@ -20,7 +20,10 @@
 <xacro:arg name="anchorZ" default="10."/>
 <xacro:arg name="wall_inclination" default="0.0"/>
-<xacro:arg name="obstacle_x" default="-0.5"/>
-<xacro:arg name="obstacle_y" default="2.5"/>
-<xacro:arg name="obstacle_z" default="-6"/>
+<xacro:arg name="obstacle_location_x" default="-0.5"/>
+<xacro:arg name="obstacle_location_y" default="2.5"/>
+<xacro:arg name="obstacle_location_z" default="-6"/>
+<xacro:arg name="obstacle_size_x" default="1.5"/>
+<xacro:arg name="obstacle_size_y" default="1.5"/>
+<xacro:arg name="obstacle_size_z" default="0.866"/>
 	<link name="wall">
 		<inertial>
@@ -74,14 +77,14 @@
   	        </inertial>
 		<visual > <!-- dont put name otherwise gazebo discards color-->
- 			  <origin rpy="0 0 0" xyz="$(arg obstacle_x) $(arg obstacle_y)  ${$(arg anchorZ) + $(arg obstacle_z)} "/>
+ 			  <origin rpy="0 0 0" xyz="$(arg obstacle_location_x) $(arg obstacle_location_y)  ${$(arg anchorZ) + $(arg obstacle_location_z)} "/>
 			<geometry>
-	                  <mesh filename="package://climbingrobot_description/meshes/ellipsoid.stl" scale="1 1 1"/>
+	                  <mesh filename="package://climbingrobot_description/meshes/ellipsoid.stl" scale="${$(arg obstacle_size_x)/1.5}  ${$(arg obstacle_size_y)/1.5}  ${$(arg obstacle_size_z)/0.866} "/>
 	                </geometry>
 			 <material name="orange"/>
 		</visual>
 		<collision>
-			<origin rpy="0 0 0" xyz="$(arg obstacle_x) $(arg obstacle_y)  ${$(arg anchorZ) + $(arg obstacle_z)} "/>
+			<origin rpy="0 0 0" xyz="$(arg obstacle_location_x) $(arg obstacle_location_y)  ${$(arg anchorZ) + $(arg obstacle_location_z)} "/>
 			 <geometry>
-	                  <mesh filename="package://climbingrobot_description/meshes/ellipsoid.stl" scale="1 1 1"/>
+	                  <mesh filename="package://climbingrobot_description/meshes/ellipsoid.stl" scale="${$(arg obstacle_size_x)/1.5}  ${$(arg obstacle_size_y)/1.5}  ${$(arg obstacle_size_z)/0.866} "/>
 	                </geometry>
 	       </collision>

Commit message: bugfix: slanted wall was not passing throught the anchor

File: urdf/climb_wall2.xacro (robot description, xacro)
@@ -32,5 +32,5 @@
   	     </inertial>
 		<visual > <!-- dont put name otherwise gazebo discards color-->
- 			<origin xyz="${$(arg anchorZ)/2 *sin($(arg wall_inclination))}  0 ${$(arg anchorZ)/2}" rpy="0  -$(arg wall_inclination) 0"/>
+ 			<origin xyz="${$(arg anchorZ)/2 *sin($(arg wall_inclination))}  0 ${$(arg anchorZ) * (1-0.5*cos($(arg wall_inclination)))}" rpy="0  -$(arg wall_inclination) 0"/>
 			<geometry>
 				<box size="0.1 $(arg anchorZ) $(arg anchorZ)"/>
@@ -39,5 +39,5 @@
 		</visual>
 	        <collision name="box">
-		       <origin xyz="${$(arg anchorZ)/2 *sin($(arg wall_inclination))} 0 ${$(arg anchorZ)/2}" rpy="0  -$(arg wall_inclination) 0"/>
+		       <origin xyz="${$(arg anchorZ)/2 *sin($(arg wall_inclination))} 0 ${$(arg anchorZ) * (1-0.5*cos($(arg wall_inclination)))}" rpy="0  -$(arg wall_inclination) 0"/>
 		       <geometry>
  				<box size="0.1 $(arg anchorZ) $(arg anchorZ)"/>
