Commit message: changes to make sumulation work with lander: increase base_link mass and moved com 5 cm lower

File: urdf/climbingrobot2landing.xacro (robot description, xacro)
@@ -13,5 +13,5 @@
    <xacro:arg name="hoist_distance" default="0.1"/>
    <xacro:arg name="hoist_base_distanceZ" default="0.05"/>
-   <xacro:arg name="lowerleg_landing_length" default="0.1"/>
+   <xacro:arg name="lowerleg_landing_length" default="0.4"/>
     <xacro:include filename="$(find climbingrobot_description)/gazebo/gazebo.urdf.xacro">
         <xacro:arg name="task_period" value="$(arg task_period)"/>
@@ -364,7 +364,7 @@
     <!-- BASE LINK INERTIAL -->
     <inertial>
-      <origin rpy="0 0 0" xyz="0 0 0"/>
+      <origin rpy="0 0 0" xyz="0 0 -0.05"/>
       <!-- <mass value="0.36"/> -->
-      <mass value="3.47"/>
+      <mass value="13.47"/>
       <!-- The base is extremely symmetrical. -->
       <inertia ixx="0.5" ixy="0.0" ixz="0.0" iyy="0.5" iyz="0.0" izz="0.5"/>

Commit message: added bumpers for lander legs

File: urdf/climbingrobot2landing.xacro (robot description, xacro)
@@ -460,4 +460,27 @@
     </collision>
    </link>
+ <gazebo reference="foot_landing_l">
+        <kp>1000000.0</kp>
+        <kd>100.0</kd>
+        <mu1>1.8</mu1>
+        <mu2>1.8</mu2>
+        <maxVel>1.0</maxVel>
+        <maxContacts>1</maxContacts>
+        <sensor name="foot_contact_sensor" type="contact">
+                <always_on>true</always_on>
+                <update_rate>1000.0</update_rate>
+                <contact>
+                <collision>lowerleg_landing_l_fixed_joint_lump__foot_landing_l_collision</collision>
+                </contact>
+                <!-- the sensor readings in terms of force torques are expressed in the lowerleg frame
+                because gazebo lumps the fake footframe with the real parent link, the normals are in the world frame-->
+                <plugin name="foot_bumper" filename="libgazebo_ros_bumper.so">
+                        <bumperTopicName>/$(arg robot_name)/foot_landing_l_bumper</bumperTopicName>
+                        <!--robotNamespace>solo</robotNamespace-->
+                        <frameName>foot_landing_l</frameName>
+                </plugin>
+        </sensor>
+        <material>Gazebo/Black</material>
+   </gazebo>
 <!--LANDING MECHANISM RIGHT-->
   <joint name="hip_yaw_landing_r" type="revolute">
@@ -526,4 +549,27 @@
     </collision>
    </link>
+    <gazebo reference="foot_landing_r">
+        <kp>1000000.0</kp>
+        <kd>100.0</kd>
+        <mu1>1.8</mu1>
+        <mu2>1.8</mu2>
+        <maxVel>1.0</maxVel>
+        <maxContacts>1</maxContacts>
+        <sensor name="foot_contact_sensor" type="contact">
+                <always_on>true</always_on>
+                <update_rate>1000.0</update_rate>
+                <contact>
+                <collision>lowerleg_landing_r_fixed_joint_lump__foot_landing_r_collision</collision>
+                </contact>
+                <!-- the sensor readings in terms of force torques are expressed in the lowerleg frame
+                because gazebo lumps the fake footframe with the real parent link, the normals are in the world frame-->
+                <plugin name="foot_bumper" filename="libgazebo_ros_bumper.so">
+                        <bumperTopicName>/$(arg robot_name)/foot_landing_r_bumper</bumperTopicName>
+                        <!--robotNamespace>solo</robotNamespace-->
+                        <frameName>foot_landing_r</frameName>
+                </plugin>
+        </sensor>
+        <material>Gazebo/Black</material>
+   </gazebo>
   <!-- Joint between the base and the ${prefix} upper leg -->
   <joint name="hip_pitch" type="revolute">

Commit message: increased mass of wheels cause sim do be unstable

File: urdf/climbingrobot2landing.xacro (robot description, xacro)
@@ -603,6 +603,6 @@
                <inertial>
                     <origin xyz="0 0 0" rpy="0 0 0"/>
-                    <mass value="0.00693606"/>
-                    <inertia ixx="0.00000057" ixy="0.0" ixz="0.0" iyy="0.00000084" iyz="0.0" izz="0.00000053"/>
+                    <mass value="0.5"/>
+                   <inertia ixx="0.00001" ixy="0.0" ixz="0.0" iyy="0.00001" iyz="0.0" izz="0.00001"/>
                 </inertial>
         </link>
@@ -636,6 +636,6 @@
                <inertial>
                     <origin xyz="0 0 0" rpy="0 0 0"/>
-                    <mass value="0.00693606"/>
-                    <inertia ixx="0.00000057" ixy="0.0" ixz="0.0" iyy="0.00000084" iyz="0.0" izz="0.00000053"/>
+                    <mass value="0.5"/>
+                    <inertia ixx="0.00001" ixy="0.0" ixz="0.0" iyy="0.00001" iyz="0.0" izz="0.00001"/>
                 </inertial>
         </link>
