Commit message: added climbingrobot2

File: urdf/climbingrobot2.xacro (robot description, xacro)
@@ -1,32 +1,22 @@
 <?xml version="1.0" ?>
-<robot name="climbingrobot" xmlns:xacro="http://ros.org/wiki/xacro">
+<robot name="climbingrobot2" xmlns:xacro="http://ros.org/wiki/xacro">
   <!-- This file is based on: https://atlas.is.localnet/confluence/display/AMDW/Quadruped+URDF+Files -->
     <!--- new_gazebo_version should be false by default because pinocchio needs it!-->
-    <xacro:arg name="robot_name" default="climbingrobot"/>
+    <xacro:arg name="robot_name" default="climbingrobot2"/>
     <xacro:arg name="new_gazebo_version" default="false"/>
-    <xacro:arg name="anchorZ" default="1."/>
+   <xacro:arg name="anchorX" default="0."/>
+   <xacro:arg name="anchorY" default="0."/>
+   <xacro:arg name="anchorZ" default="1."/>
+   <xacro:arg name="anchor2X" default="0."/>
+   <xacro:arg name="anchor2Y" default="0."/>
+   <xacro:arg name="anchor2Z" default="1."/>
     <xacro:include filename="$(find climbingrobot_description)/gazebo/gazebo.urdf.xacro">
         <xacro:arg name="task_period" value="$(arg task_period)"/>
 	<xacro:arg name="robot_name" value="$(arg robot_name)"/>
     </xacro:include>
-    <xacro:include filename="$(find climbingrobot_description)/urdf/climbingrobot.transmission.xacro"/>
-    <link name="world"/>
-   <joint name="mountain" type="fixed">
-        <origin rpy="0 0 0" xyz="0 0 $(arg anchorZ)"/>
-        <parent link="world"/>
-        <child link="anchor"/>
-    </joint>
-    <link name="anchor">
-    <visual>
-	<geometry>
-         <sphere radius="0.4" />
-	</geometry>
-    </visual>
-    <inertial>
-      <origin rpy="0 0 0" xyz="0 0 0.0"/>
-      <mass value="0.01"/>
-      <inertia ixx="0.01" ixy="0.0" ixz="0.0" iyy="0.01" iyz="0.0" izz="0.01"/>
-    </inertial>
-  </link>
+    <xacro:include filename="$(find climbingrobot_description)/urdf/climbingrobot2.transmission.xacro"/>
+ <material name="Blue">
+    <color rgba="${0/255} ${0/255} ${255/255} 1.0"/>
+  </material>
 <!--
     <joint name="target_link" type="fixed">
@@ -48,4 +38,23 @@
     </inertial>
   </link>-->
+    <link name="world"/>
+ <!-- Anchor 1-->
+   <joint name="anchor1_position" type="fixed">
+        <origin rpy="0 0 0" xyz="$(arg anchorX) $(arg anchorY) $(arg anchorZ)"/>
+        <parent link="world"/>
+        <child link="anchor"/>
+    </joint>
+    <link name="anchor">
+    <visual>
+	<geometry>
+         <sphere radius="0.4" />
+	</geometry>
+    </visual>
+    <inertial>
+      <origin rpy="0 0 0" xyz="0 0 0.0"/>
+      <mass value="0.01"/>
+      <inertia ixx="0.01" ixy="0.0" ixz="0.0" iyy="0.01" iyz="0.0" izz="0.01"/>
+    </inertial>
+  </link>
   <!-- Revolute pitch joint between the mountain and the wire -->
   <joint name="mountain_wire_pitch" type="revolute">
@@ -164,4 +173,287 @@
     <dynamics damping="0.0" friction="0.0"/>
   </joint>
+  <!-- Anchor 2 closed loop kinematics Gazebo -->
+  <xacro:if value="$(arg new_gazebo_version)">
+   <joint name="anchor2_position" type="fixed">
+        <origin rpy="0 0 0" xyz="$(arg anchor2X) $(arg anchor2Y) 0"/>
+        <parent link="anchor"/>
+        <child link="anchor_2"/>
+    </joint>
+    <link name="anchor_2">
+	    <visual>
+		<geometry>
+		 <sphere radius="0.4" />
+		</geometry>
+		<material name="Blue"/><!--rviz"/-->
+	    </visual>
+	    <inertial>
+	      <origin rpy="0 0 0" xyz="0 0 0.0"/>
+	      <mass value="0.01"/>
+	      <inertia ixx="0.01" ixy="0.0" ixz="0.0" iyy="0.01" iyz="0.0" izz="0.01"/>
+	    </inertial>
+    </link>
+  <!-- Revolute pitch joint between the mountain and the wire -->
+  <joint name="mountain_wire_pitch_2" type="revolute">
+    <parent link="anchor_2"/>
+    <child link="pre_wire1_2"/>
+    <limit effort="1000" velocity="100.0" lower="-100" upper="100"/>
+    <!-- joint rotates about -y axis -->
+    <axis xyz="0 -1 0"/>
+    <origin rpy="0 0 0" xyz="0.0 0.0 0.0"/>
+    <!-- pybullet simulation parameters -->
+    <dynamics damping="0.0" friction="0.0"/>
+  </joint>
+  <link name="pre_wire1_2">
+    <visual>
+      <origin rpy="0 0 0" xyz="0 0 0"/>
+      <geometry>
+        <mesh filename="package://climbingrobot_description/meshes/obj/cylinder.obj" scale="0.01 0.01 0.01"/>
+      </geometry>
+      <material name="grey">
+        <color rgba=".7 .7 .7 .5"/>
+      </material>
+    </visual>
+    <collision>
+      <origin rpy="0 0 0" xyz="0 0 0.0"/>
+      <geometry>
+        <cylinder length="0.01" radius="0.01"/>
+      </geometry>
+    </collision>
+    <inertial>
+      <origin rpy="0 0 0" xyz="0 0 0.0"/>
+      <mass value="0.01"/>
+      <inertia ixx="0.0001" ixy="0.0" ixz="0.0" iyy="0.0001" iyz="0.0" izz="0.0001"/>
+    </inertial>
+  </link>
+  <!-- Revolute roll joint between the mountain and the wire -->
+  <joint name="mountain_wire_roll_2" type="revolute">
+    <parent link="pre_wire1_2"/>
+    <child link="wire_2"/>
+    <limit effort="1000" velocity="100.0" lower="-100" upper="100"/>
+    <!-- joint rotates about x axis -->
+    <axis xyz="1 0 0"/>
+    <origin rpy="0 0 0" xyz="0.0 0.0 0.0"/>
+    <!-- pybullet simulation parameters -->
+    <dynamics damping="0.0" friction="0.0"/>
+  </joint>
+  <link name="wire_2">
+    <inertial>
+      <origin rpy="0 0 0" xyz="0 0 0.0"/>
+      <mass value="0.01"/>
+      <inertia ixx="0.001" ixy="0.0" ixz="0.0" iyy="0.001" iyz="0.0" izz="0.001"/>
+    </inertial>
+  </link>
+  <!-- Prismatic joint between the wire and the base -->
+  <joint name="wire_base_prismatic_2" type="prismatic">
+    <parent link="wire_2"/>
+    <child link="pre-base1_2"/>
+    <limit effort="1000" velocity="100.0" lower="-100" upper="100"/>
+    <!-- joint translates on x axis -->
+    <axis xyz="0 0 -1"/>
+    <origin rpy="0 0 0" xyz="0.0 0.0 0.0"/>
+    <!-- pybullet simulation parameters -->
+    <dynamics damping="0.0" friction="0.0"/>
+  </joint>
+  <link name="pre-base1_2">
+    <inertial>
+      <origin rpy="0 0 0" xyz="0 0 0.0"/>
+      <mass value="0.01"/>
+      <inertia ixx="0.0001" ixy="0.0" ixz="0.0" iyy="0.0001" iyz="0.0" izz="0.0001"/>
+    </inertial>
+  </link>
+  <!-- Revolute pitch joint between the wire and the base -->
+  <joint name="wire_base_pitch_2" type="revolute">
+    <parent link="pre-base1_2"/>
+    <child link="pre-base2_2"/>
+    <limit effort="1000" velocity="100.0" lower="-100" upper="100"/>
+    <!-- joint rotates about y axis -->
+    <axis xyz="0 1 0"/>
+    <origin rpy="0 0 0" xyz="0.0 0.0 0.0"/>
+    <!-- pybullet simulation parameters -->
+    <dynamics damping="0.0" friction="0.0"/>
+  </joint>
+  <link name="pre-base2_2">
+     <inertial>
+      <origin rpy="0 0 0" xyz="0 0 0.0"/>
+      <mass value="0.01"/>
+      <inertia ixx="0.0001" ixy="0.0" ixz="0.0" iyy="0.0001" iyz="0.0" izz="0.0001"/>
+    </inertial>
+  </link>
+  <!-- Revolute roll joint between the wire and the base -->
+  <joint name="wire_base_roll_2" type="revolute">
+    <parent link="pre-base2_2"/>
+    <child link="pre-base3_2"/>
+    <limit effort="1000" velocity="100.0" lower="-100" upper="100"/>
+    <!-- joint rotates about x axis -->
+    <axis xyz="1 0 0"/>
+    <origin rpy="0 0 0" xyz="0.0 0.0 0.0"/>
+    <!-- pybullet simulation parameters -->
+    <dynamics damping="0.0" friction="0.0"/>
+  </joint>
+  <link name="pre-base3_2">
+    <inertial>
+      <origin rpy="0 0 0" xyz="0 0 0.0"/>
+      <mass value="0.01"/>
+      <inertia ixx="0.0001" ixy="0.0" ixz="0.0" iyy="0.0001" iyz="0.0" izz="0.0001"/>
+    </inertial>
+  </link>
+  <!-- Revolute yaw joint between the wire and the base -->
+  <joint name="wire_base_yaw_2" type="revolute">
+    <parent link="pre-base3_2"/>
+    <child link="fake_connection"/>
+    <limit effort="1000" velocity="100.0" lower="-100" upper="100"/>
+    <!-- joint rotates about z axis -->
+    <axis xyz="0 0 1"/>
+    <origin rpy="0 0 0" xyz="0.0 0.0 0.0"/>
+    <!-- pybullet simulation parameters -->
+    <dynamics damping="0.0" friction="0.0"/>
+  </joint>
+  <link name="fake_connection">
+    <inertial>
+      <origin rpy="0 0 0" xyz="0 0 0.0"/>
+      <mass value="0.001"/>
+      <inertia ixx="0.00001" ixy="0.0" ixz="0.0" iyy="0.00001" iyz="0.0" izz="0.00001"/>
+    </inertial>
+  </link>
+	<gazebo>
+	    <joint name="connection_to_base_link" type="fixed">
+	      <pose>0 0 0 0 0 0 0</pose>
+	      <parent>fake_connection</parent>
+	      <child>base_link</child>
+	    </joint>
+	</gazebo>
+ </xacro:if>
+<!-- Anchor 2 open loop kinematics Pinocchio-->
+  <xacro:unless value="$(arg new_gazebo_version)">
+  <!-- Revolute yaw joint between the wire and the base -->
+  <joint name="wire_base_yaw_2" type="revolute">
+    <parent link="base_link"/>
+    <child link="pre-base3_2"/>
+    <limit effort="1000" velocity="100.0" lower="-100" upper="100"/>
+    <!-- joint rotates about z axis -->
+    <axis xyz="0 0 1"/>
+    <origin rpy="0 0 0" xyz="0.0 0.0 0.0"/>
+    <!-- pybullet simulation parameters -->
+    <dynamics damping="0.0" friction="0.0"/>
+  </joint>
+  <link name="pre-base3_2">
+    <inertial>
+      <origin rpy="0 0 0" xyz="0 0 0.0"/>
+      <mass value="0.01"/>
+      <inertia ixx="0.0001" ixy="0.0" ixz="0.0" iyy="0.0001" iyz="0.0" izz="0.0001"/>
+    </inertial>
+  </link>
+  <!-- Revolute roll joint between the wire and the base -->
+  <joint name="wire_base_roll_2" type="revolute">
+    <parent link="pre-base3_2"/>
+    <child link="pre-base2_2"/>
+    <limit effort="1000" velocity="100.0" lower="-100" upper="100"/>
+    <!-- joint rotates about x axis -->
+    <axis xyz="1 0 0"/>
+    <origin rpy="0 0 0" xyz="0.0 0.0 0.0"/>
+    <!-- pybullet simulation parameters -->
+    <dynamics damping="0.0" friction="0.0"/>
+  </joint>
+  <link name="pre-base2_2">
+     <inertial>
+      <origin rpy="0 0 0" xyz="0 0 0.0"/>
+      <mass value="0.01"/>
+      <inertia ixx="0.0001" ixy="0.0" ixz="0.0" iyy="0.0001" iyz="0.0" izz="0.0001"/>
+    </inertial>
+  </link>
+  <!-- Revolute pitch joint between the wire and the base -->
+  <joint name="wire_base_pitch_2" type="revolute">
+    <parent link="pre-base2_2"/>
+    <child link="pre-base1_2"/>
+    <limit effort="1000" velocity="100.0" lower="-100" upper="100"/>
+    <!-- joint rotates about y axis -->
+    <axis xyz="0 1 0"/>
+    <origin rpy="0 0 0" xyz="0.0 0.0 0.0"/>
+    <!-- pybullet simulation parameters -->
+    <dynamics damping="0.0" friction="0.0"/>
+  </joint>
+    <link name="pre-base1_2">
+    <inertial>
+      <origin rpy="0 0 0" xyz="0 0 0.0"/>
+      <mass value="0.01"/>
+      <inertia ixx="0.0001" ixy="0.0" ixz="0.0" iyy="0.0001" iyz="0.0" izz="0.0001"/>
+    </inertial>
+  </link>
+<!-- Prismatic joint between the wire and the base -->
+  <joint name="wire_base_prismatic_2" type="prismatic">
+    <parent link="pre-base1_2"/>
+    <child link="wire_2"/>
+    <limit effort="1000" velocity="100.0" lower="-100" upper="100"/>
+    <!-- joint translates on x axis -->
+    <axis xyz="0 0 -1"/>
+    <origin rpy="0 0 0" xyz="0.0 0.0 0.0"/>
+    <!-- pybullet simulation parameters -->
+    <dynamics damping="0.0" friction="0.0"/>
+  </joint>
+  <link name="wire_2">
+    <inertial>
+      <origin rpy="0 0 0" xyz="0 0 0.0"/>
+      <mass value="0.01"/>
+      <inertia ixx="0.001" ixy="0.0" ixz="0.0" iyy="0.001" iyz="0.0" izz="0.001"/>
+    </inertial>
+  </link>
+  <!-- Revolute roll joint between the mountain and the wire -->
+  <joint name="mountain_wire_roll_2" type="revolute">
+    <parent link="wire_2"/>
+    <child link="pre_wire1_2"/>
+    <limit effort="1000" velocity="100.0" lower="-100" upper="100"/>
+    <!-- joint rotates about x axis -->
+    <axis xyz="1 0 0"/>
+    <origin rpy="0 0 0" xyz="0.0 0.0 0.0"/>
+    <!-- pybullet simulation parameters -->
+    <dynamics damping="0.0" friction="0.0"/>
+  </joint>
+<link name="pre_wire1_2">
+    <visual>
+      <origin rpy="0 0 0" xyz="0 0 0"/>
+      <geometry>
+        <mesh filename="package://climbingrobot_description/meshes/obj/cylinder.obj" scale="0.01 0.01 0.01"/>
+      </geometry>
+      <material name="grey">
+        <color rgba=".7 .7 .7 .5"/>
+      </material>
+    </visual>
+    <collision>
+      <origin rpy="0 0 0" xyz="0 0 0.0"/>
+      <geometry>
+        <cylinder length="0.01" radius="0.01"/>
+      </geometry>
+    </collision>
+    <inertial>
+      <origin rpy="0 0 0" xyz="0 0 0.0"/>
+      <mass value="0.01"/>
+      <inertia ixx="0.0001" ixy="0.0" ixz="0.0" iyy="0.0001" iyz="0.0" izz="0.0001"/>
+    </inertial>
+  </link>
+<!-- Revolute pitch joint between the mountain and the wire -->
+  <joint name="mountain_wire_pitch_2" type="revolute">
+    <parent link="pre_wire1_2"/>
+    <child link="anchor_2"/>
+    <limit effort="1000" velocity="100.0" lower="-100" upper="100"/>
+    <!-- joint rotates about -y axis -->
+    <axis xyz="0 -1 0"/>
+    <origin rpy="0 0 0" xyz="0.0 0.0 0.0"/>
+    <!-- pybullet simulation parameters -->
+    <dynamics damping="0.0" friction="0.0"/>
+  </joint>
+ <link name="anchor_2">
+	    <visual>
+		<geometry>
+		 <sphere radius="0.5" />
+		</geometry>
+		<material name="Blue"/><!--rviz"/-->
+	    </visual>
+	    <inertial>
+	      <origin rpy="0 0 0" xyz="0 0 0.0"/>
+	      <mass value="0.01"/>
+	      <inertia ixx="0.01" ixy="0.0" ixz="0.0" iyy="0.01" iyz="0.0" izz="0.01"/>
+	    </inertial>
+    </link>
+ </xacro:unless>
   <link name="base_link">
     <!-- BASE LINK INERTIAL -->

Commit message: cutting the kin loop in the same place for pinocchio and gazebo

File: urdf/climbingrobot2.xacro (robot description, xacro)
@@ -174,5 +174,4 @@
   </joint>
   <!-- Anchor 2 closed loop kinematics Gazebo -->
-  <xacro:if value="$(arg new_gazebo_version)">
    <joint name="anchor2_position" type="fixed">
         <origin rpy="0 0 0" xyz="$(arg anchor2X) $(arg anchor2Y) 0"/>
@@ -316,4 +315,5 @@
     </inertial>
   </link>
+  <xacro:if value="$(arg new_gazebo_version)">
 	<gazebo>
 	    <joint name="connection_to_base_link" type="fixed">
@@ -324,136 +324,4 @@
 	</gazebo>
  </xacro:if>
-<!-- Anchor 2 open loop kinematics Pinocchio-->
-  <xacro:unless value="$(arg new_gazebo_version)">
-  <!-- Revolute yaw joint between the wire and the base -->
-  <joint name="wire_base_yaw_2" type="revolute">
-    <parent link="base_link"/>
-    <child link="pre-base3_2"/>
-    <limit effort="1000" velocity="100.0" lower="-100" upper="100"/>
-    <!-- joint rotates about z axis -->
-    <axis xyz="0 0 1"/>
-    <origin rpy="0 0 0" xyz="0.0 0.0 0.0"/>
-    <!-- pybullet simulation parameters -->
-    <dynamics damping="0.0" friction="0.0"/>
-  </joint>
-  <link name="pre-base3_2">
-    <inertial>
-      <origin rpy="0 0 0" xyz="0 0 0.0"/>
-      <mass value="0.01"/>
-      <inertia ixx="0.0001" ixy="0.0" ixz="0.0" iyy="0.0001" iyz="0.0" izz="0.0001"/>
-    </inertial>
-  </link>
-  <!-- Revolute roll joint between the wire and the base -->
-  <joint name="wire_base_roll_2" type="revolute">
-    <parent link="pre-base3_2"/>
-    <child link="pre-base2_2"/>
-    <limit effort="1000" velocity="100.0" lower="-100" upper="100"/>
-    <!-- joint rotates about x axis -->
-    <axis xyz="1 0 0"/>
-    <origin rpy="0 0 0" xyz="0.0 0.0 0.0"/>
-    <!-- pybullet simulation parameters -->
-    <dynamics damping="0.0" friction="0.0"/>
-  </joint>
-  <link name="pre-base2_2">
-     <inertial>
-      <origin rpy="0 0 0" xyz="0 0 0.0"/>
-      <mass value="0.01"/>
-      <inertia ixx="0.0001" ixy="0.0" ixz="0.0" iyy="0.0001" iyz="0.0" izz="0.0001"/>
-    </inertial>
-  </link>
-  <!-- Revolute pitch joint between the wire and the base -->
-  <joint name="wire_base_pitch_2" type="revolute">
-    <parent link="pre-base2_2"/>
-    <child link="pre-base1_2"/>
-    <limit effort="1000" velocity="100.0" lower="-100" upper="100"/>
-    <!-- joint rotates about y axis -->
-    <axis xyz="0 1 0"/>
-    <origin rpy="0 0 0" xyz="0.0 0.0 0.0"/>
-    <!-- pybullet simulation parameters -->
-    <dynamics damping="0.0" friction="0.0"/>
-  </joint>
-    <link name="pre-base1_2">
-    <inertial>
-      <origin rpy="0 0 0" xyz="0 0 0.0"/>
-      <mass value="0.01"/>
-      <inertia ixx="0.0001" ixy="0.0" ixz="0.0" iyy="0.0001" iyz="0.0" izz="0.0001"/>
-    </inertial>
-  </link>
-<!-- Prismatic joint between the wire and the base -->
-  <joint name="wire_base_prismatic_2" type="prismatic">
-    <parent link="pre-base1_2"/>
-    <child link="wire_2"/>
-    <limit effort="1000" velocity="100.0" lower="-100" upper="100"/>
-    <!-- joint translates on x axis -->
-    <axis xyz="0 0 -1"/>
-    <origin rpy="0 0 0" xyz="0.0 0.0 0.0"/>
-    <!-- pybullet simulation parameters -->
-    <dynamics damping="0.0" friction="0.0"/>
-  </joint>
-  <link name="wire_2">
-    <inertial>
-      <origin rpy="0 0 0" xyz="0 0 0.0"/>
-      <mass value="0.01"/>
-      <inertia ixx="0.001" ixy="0.0" ixz="0.0" iyy="0.001" iyz="0.0" izz="0.001"/>
-    </inertial>
-  </link>
-  <!-- Revolute roll joint between the mountain and the wire -->
-  <joint name="mountain_wire_roll_2" type="revolute">
-    <parent link="wire_2"/>
-    <child link="pre_wire1_2"/>
-    <limit effort="1000" velocity="100.0" lower="-100" upper="100"/>
-    <!-- joint rotates about x axis -->
-    <axis xyz="1 0 0"/>
-    <origin rpy="0 0 0" xyz="0.0 0.0 0.0"/>
-    <!-- pybullet simulation parameters -->
-    <dynamics damping="0.0" friction="0.0"/>
-  </joint>
-<link name="pre_wire1_2">
-    <visual>
-      <origin rpy="0 0 0" xyz="0 0 0"/>
-      <geometry>
-        <mesh filename="package://climbingrobot_description/meshes/obj/cylinder.obj" scale="0.01 0.01 0.01"/>
-      </geometry>
-      <material name="grey">
-        <color rgba=".7 .7 .7 .5"/>
-      </material>
-    </visual>
-    <collision>
-      <origin rpy="0 0 0" xyz="0 0 0.0"/>
-      <geometry>
-        <cylinder length="0.01" radius="0.01"/>
-      </geometry>
-    </collision>
-    <inertial>
-      <origin rpy="0 0 0" xyz="0 0 0.0"/>
-      <mass value="0.01"/>
-      <inertia ixx="0.0001" ixy="0.0" ixz="0.0" iyy="0.0001" iyz="0.0" izz="0.0001"/>
-    </inertial>
-  </link>
-<!-- Revolute pitch joint between the mountain and the wire -->
-  <joint name="mountain_wire_pitch_2" type="revolute">
-    <parent link="pre_wire1_2"/>
-    <child link="anchor_2"/>
-    <limit effort="1000" velocity="100.0" lower="-100" upper="100"/>
-    <!-- joint rotates about -y axis -->
-    <axis xyz="0 -1 0"/>
-    <origin rpy="0 0 0" xyz="0.0 0.0 0.0"/>
-    <!-- pybullet simulation parameters -->
-    <dynamics damping="0.0" friction="0.0"/>
-  </joint>
- <link name="anchor_2">
-	    <visual>
-		<geometry>
-		 <sphere radius="0.5" />
-		</geometry>
-		<material name="Blue"/><!--rviz"/-->
-	    </visual>
-	    <inertial>
-	      <origin rpy="0 0 0" xyz="0 0 0.0"/>
-	      <mass value="0.01"/>
-	      <inertia ixx="0.01" ixy="0.0" ixz="0.0" iyy="0.01" iyz="0.0" izz="0.01"/>
-	    </inertial>
-    </link>
- </xacro:unless>
   <link name="base_link">
     <!-- BASE LINK INERTIAL -->

Commit message: cutting the loop in a different place to do not have 2 joints have the same child base link (fixed link on anchor 2 wrt anchor)

File: urdf/climbingrobot2.xacro (robot description, xacro)
@@ -120,4 +120,22 @@
   </joint>
   <link name="pre-base1">
+      <visual>
+      <origin rpy="0 0 0" xyz="0 0 ${$(arg anchorZ)/2}"/>
+     <geometry>
+           <cylinder radius="0.05" length="$(arg anchorZ)"/>
+      </geometry>
+ 	      <material name="grey">
+ 	        <color rgba=".7 .7 .7 .5"/>
+ 	      </material>
+     </visual>
+     <collision>
+ 	      <origin rpy="0 0 0" xyz="0 0 $(arg anchorZ)"/>
+ 	      <geometry>
+ 	        <cylinder radius="0.05" length="${$(arg anchorZ)*2}"/>
+ 	      </geometry>
+ 	      <material name="grey">
+ 	        <color rgba=".7 .7 .7 .5"/>
+ 	      </material>
+    </collision>
     <inertial>
       <origin rpy="0 0 0" xyz="0 0 0.0"/>
@@ -173,5 +191,5 @@
     <dynamics damping="0.0" friction="0.0"/>
   </joint>
-  <!-- Anchor 2 closed loop kinematics Gazebo -->
+  <!-- Anchor 2   -->
    <joint name="anchor2_position" type="fixed">
         <origin rpy="0 0 0" xyz="$(arg anchor2X) $(arg anchor2Y) 0"/>
@@ -255,4 +273,22 @@
   </joint>
   <link name="pre-base1_2">
+      <visual>
+       	      <origin rpy="0 0 0" xyz="0 0 $(arg anchorZ)"/>
+ 	      <geometry>
+ 	        <cylinder radius="0.05" length="${$(arg anchorZ)*2}"/>
+ 	      </geometry>
+ 	      <material name="grey">
+ 	        <color rgba=".7 .7 .7 .5"/>
+ 	      </material>
+     </visual>
+     <collision>
+ 	      <origin rpy="0 0 0" xyz="0 0 ${$(arg anchorZ)/2}"/>
+ 	      <geometry>
+ 	        <cylinder radius="0.05" length="$(arg anchorZ)"/>
+ 	      </geometry>
+ 	      <material name="grey">
+ 	        <color rgba=".7 .7 .7 .5"/>
+ 	      </material>
+    </collision>
     <inertial>
       <origin rpy="0 0 0" xyz="0 0 0.0"/>
@@ -311,17 +347,18 @@
     <inertial>
       <origin rpy="0 0 0" xyz="0 0 0.0"/>
-      <mass value="0.001"/>
-      <inertia ixx="0.00001" ixy="0.0" ixz="0.0" iyy="0.00001" iyz="0.0" izz="0.00001"/>
-    </inertial>
-  </link>
-  <xacro:if value="$(arg new_gazebo_version)">
-	<gazebo>
-	    <joint name="connection_to_base_link" type="fixed">
-	      <pose>0 0 0 0 0 0 0</pose>
-	      <parent>fake_connection</parent>
-	      <child>base_link</child>
-	    </joint>
-	</gazebo>
- </xacro:if>
+      <mass value="0.01"/>
+      <inertia ixx="0.001" ixy="0.0" ixz="0.0" iyy="0.001" iyz="0.0" izz="0.001"/>
+    </inertial>
+  </link>
+ <!-- closing the loop for gazebo not used by pinocchio -->
+ <gazebo>
+  <joint name="fixed_joint" type="fixed">
+         <pose>0 0 0 0 0 0 0</pose>
+       <parent>fake_connection</parent>
+	 <child>base_link</child>
+ 	<axis>
+    </axis>
+  </joint>
+ </gazebo>
   <link name="base_link">
     <!-- BASE LINK INERTIAL -->

Commit message: improved q0 in climbing robot 2 to start in the middle of 2 anchors

File: urdf/climbingrobot2.xacro (robot description, xacro)
@@ -9,5 +9,5 @@
    <xacro:arg name="anchorZ" default="20."/>
    <xacro:arg name="anchor2X" default="0."/>
-   <xacro:arg name="anchor2Y" default="0."/>
+   <xacro:arg name="anchor2Y" default="5."/>
    <xacro:arg name="anchor2Z" default="20."/>
     <xacro:include filename="$(find climbingrobot_description)/gazebo/gazebo.urdf.xacro">
@@ -97,5 +97,5 @@
     <!-- joint rotates about x axis -->
     <axis xyz="1 0 0"/>
-    <origin rpy="0 0 0" xyz="0.0 0.0 0.0"/>
+    <origin rpy="1.57 0 0" xyz="0.0 0.0 0.0"/>
     <!-- pybullet simulation parameters -->
     <dynamics damping="0.0" friction="0.0"/>
@@ -115,5 +115,5 @@
     <!-- joint translates on z axis -->
     <axis xyz="0 0 -1"/>
-    <origin rpy="0 0 0" xyz="0.0 0.0 0.0"/>
+    <origin rpy="0 0 0" xyz="0.0 0.0 -${$(arg anchor2Y)/2}"/>
     <!-- pybullet simulation parameters -->
     <dynamics damping="0.0" friction="0.0"/>
@@ -268,5 +268,5 @@
     <!-- joint translates on x axis -->
     <axis xyz="0 0 -1"/>
-    <origin rpy="0 0 0" xyz="0.0 0.0 -$(arg anchor2Y)"/>
+    <origin rpy="0 0 0" xyz="0.0 0.0 -${$(arg anchor2Y)/2}"/>
     <!-- pybullet simulation parameters -->
     <dynamics damping="0.0" friction="0.0"/>
