Commit message: fixing fake link orientation to be aligned with base frame at q0

File: urdf/climbingrobot2.xacro (robot description, xacro)
@@ -339,5 +339,5 @@
     <!-- joint rotates about x axis -->
     <axis xyz="0 0 1"/>
-    <origin rpy="1.57 0 0" xyz="0.0 0.0 0.0"/>
+    <origin rpy="0 0 0" xyz="0.0 0.0 0.0"/>
     <!-- pybullet simulation parameters -->
     <dynamics damping="0.0" friction="0.0"/>

Commit message: base is now vertical at q0

File: urdf/climbingrobot2.xacro (robot description, xacro)
@@ -169,5 +169,5 @@
     <!-- joint rotates about x axis -->
     <axis xyz="1 0 0"/>
-    <origin rpy="0 0 0" xyz="0.0 0.0 0.0"/>
+    <origin rpy="-1.57 0 0" xyz="0.0 0.0 0.0"/>
     <!-- pybullet simulation parameters -->
     <dynamics damping="0.0" friction="0.0"/>
@@ -322,5 +322,5 @@
     <!-- joint rotates about x axis -->
     <axis xyz="1 0 0"/>
-    <origin rpy="0 0 0" xyz="0.0 0.0 0.0"/>
+    <origin rpy="1.57 0 0" xyz="0.0 0.0 0.0"/>
     <!-- pybullet simulation parameters -->
     <dynamics damping="0.0" friction="0.0"/>

Commit message: adding 5 cm offset between 2 joists it starts up better (also works without this need to tune low pd gains for the wire_base joints)

File: urdf/climbingrobot2.xacro (robot description, xacro)
@@ -115,5 +115,5 @@
     <!-- joint translates on z axis -->
     <axis xyz="0 0 -1"/>
-    <origin rpy="0 0 0" xyz="0.0 0.0 -${$(arg anchor2Y)/2}"/>
+    <origin rpy="0 0 0" xyz="0.0 0.0 ${0.05 -$(arg anchor2Y)/2}"/>
     <!-- pybullet simulation parameters -->
     <dynamics damping="0.0" friction="0.0"/>
@@ -187,5 +187,5 @@
     <!-- joint rotates about z axis -->
     <axis xyz="0 0 1"/>
-    <origin rpy="0 0 0" xyz="0.0 0.0 0.0"/>
+    <origin rpy="0 0 0" xyz="0.0 0.05 0.0"/>
     <!-- pybullet simulation parameters -->
     <dynamics damping="0.0" friction="0.0"/>
@@ -268,5 +268,5 @@
     <!-- joint translates on x axis -->
     <axis xyz="0 0 -1"/>
-    <origin rpy="0 0 0" xyz="0.0 0.0 -${$(arg anchor2Y)/2}"/>
+    <origin rpy="0 0 0" xyz="0.0 0.0  ${0.05 -$(arg anchor2Y)/2}"/>
     <!-- pybullet simulation parameters -->
     <dynamics damping="0.0" friction="0.0"/>
@@ -353,5 +353,5 @@
  <gazebo>
 	  <joint name="fixed_joint" type="fixed">
-		 <pose>0 0 0 0 0 0 0</pose>
+		 <pose>0 0.05 0 0 0 0 0</pose>
 		 <parent>fake_link</parent>
 		 <child>base_link</child>

Commit message: resized rope diameter

File: urdf/climbingrobot2.xacro (robot description, xacro)
@@ -125,5 +125,5 @@
       <origin rpy="0 0 0" xyz="0 0 ${$(arg anchorZ)/2}"/>
      <geometry>
-           <cylinder radius="0.05" length="$(arg anchorZ)"/>
+           <cylinder radius="0.01" length="$(arg anchorZ)"/> <!--this is the rope-->
       </geometry>
  	      <material name="grey">
@@ -134,5 +134,5 @@
  	      <origin rpy="0 0 0" xyz="0 0 $(arg anchorZ)"/>
  	      <geometry>
- 	        <cylinder radius="0.05" length="${$(arg anchorZ)*2}"/>
+ 	        <cylinder radius="0.01" length="${$(arg anchorZ)*2}"/>
  	      </geometry>
  	      <material name="grey">
@@ -278,5 +278,5 @@
        	      <origin rpy="0 0 0" xyz="0 0 $(arg anchorZ)"/>
  	      <geometry>
- 	        <cylinder radius="0.05" length="${$(arg anchorZ)*2}"/>
+ 	        <cylinder radius="0.01" length="${$(arg anchorZ)*2}"/> <!--this is the rope-->
  	      </geometry>
  	      <material name="grey">
@@ -287,5 +287,5 @@
  	      <origin rpy="0 0 0" xyz="0 0 ${$(arg anchorZ)/2}"/>
  	      <geometry>
- 	        <cylinder radius="0.05" length="$(arg anchorZ)"/>
+ 	        <cylinder radius="0.01" length="$(arg anchorZ)"/>
  	      </geometry>
  	      <material name="grey">

File: urdf/climbingrobot2landing.xacro (robot description, xacro)
@@ -127,5 +127,5 @@
       <origin rpy="0 0 0" xyz="0 0 ${$(arg anchorZ)/2}"/>
      <geometry>
-           <cylinder radius="0.05" length="$(arg anchorZ)"/>
+           <cylinder radius="0.01" length="$(arg anchorZ)"/>
       </geometry>
  	      <material name="grey">
@@ -136,5 +136,5 @@
  	      <origin rpy="0 0 0" xyz="0 0 $(arg anchorZ)"/>
  	      <geometry>
- 	        <cylinder radius="0.05" length="${$(arg anchorZ)*2}"/>
+ 	        <cylinder radius="0.01" length="${$(arg anchorZ)*2}"/>
  	      </geometry>
  	      <material name="grey">
@@ -280,5 +280,5 @@
        	      <origin rpy="0 0 0" xyz="0 0 $(arg anchorZ)"/>
  	      <geometry>
- 	        <cylinder radius="0.05" length="${$(arg anchorZ)*2}"/>
+ 	        <cylinder radius="0.01" length="${$(arg anchorZ)*2}"/>
  	      </geometry>
  	      <material name="grey">
@@ -289,5 +289,5 @@
  	      <origin rpy="0 0 0" xyz="0 0 ${$(arg anchorZ)/2}"/>
  	      <geometry>
- 	        <cylinder radius="0.05" length="$(arg anchorZ)"/>
+ 	        <cylinder radius="0.01" length="$(arg anchorZ)"/>
  	      </geometry>
  	      <material name="grey">

Commit message: increasing rope size for paper

File: urdf/climbingrobot2.xacro (robot description, xacro)
@@ -125,5 +125,5 @@
       <origin rpy="0 0 0" xyz="0 0 ${$(arg anchorZ)/2}"/>
      <geometry>
-           <cylinder radius="0.01" length="$(arg anchorZ)"/> <!--this is the rope-->
+           <cylinder radius="0.025" length="$(arg anchorZ)"/> <!--this is the rope-->
       </geometry>
  	      <material name="grey">
@@ -134,5 +134,5 @@
  	      <origin rpy="0 0 0" xyz="0 0 $(arg anchorZ)"/>
  	      <geometry>
- 	        <cylinder radius="0.01" length="${$(arg anchorZ)*2}"/>
+ 	        <cylinder radius="0.025" length="${$(arg anchorZ)*2}"/>
  	      </geometry>
  	      <material name="grey">
@@ -278,5 +278,5 @@
        	      <origin rpy="0 0 0" xyz="0 0 $(arg anchorZ)"/>
  	      <geometry>
- 	        <cylinder radius="0.01" length="${$(arg anchorZ)*2}"/> <!--this is the rope-->
+ 	        <cylinder radius="0.025" length="${$(arg anchorZ)*2}"/> <!--this is the rope-->
  	      </geometry>
  	      <material name="grey">
@@ -287,5 +287,5 @@
  	      <origin rpy="0 0 0" xyz="0 0 ${$(arg anchorZ)/2}"/>
  	      <geometry>
- 	        <cylinder radius="0.01" length="$(arg anchorZ)"/>
+ 	        <cylinder radius="0.025" length="$(arg anchorZ)"/>
  	      </geometry>
  	      <material name="grey">

File: urdf/climbingrobot2landing.xacro (robot description, xacro)
@@ -127,5 +127,5 @@
       <origin rpy="0 0 0" xyz="0 0 ${$(arg anchorZ)/2}"/>
      <geometry>
-           <cylinder radius="0.01" length="$(arg anchorZ)"/>
+           <cylinder radius="0.025" length="$(arg anchorZ)"/><!--this is the rope-->
       </geometry>
  	      <material name="grey">
@@ -136,5 +136,5 @@
  	      <origin rpy="0 0 0" xyz="0 0 $(arg anchorZ)"/>
  	      <geometry>
- 	        <cylinder radius="0.01" length="${$(arg anchorZ)*2}"/>
+ 	        <cylinder radius="0.025" length="${$(arg anchorZ)*2}"/>
  	      </geometry>
  	      <material name="grey">
@@ -280,5 +280,5 @@
        	      <origin rpy="0 0 0" xyz="0 0 $(arg anchorZ)"/>
  	      <geometry>
- 	        <cylinder radius="0.01" length="${$(arg anchorZ)*2}"/>
+ 	        <cylinder radius="0.025" length="${$(arg anchorZ)*2}"/><!--this is the rope-->
  	      </geometry>
  	      <material name="grey">
@@ -289,5 +289,5 @@
  	      <origin rpy="0 0 0" xyz="0 0 ${$(arg anchorZ)/2}"/>
  	      <geometry>
- 	        <cylinder radius="0.01" length="$(arg anchorZ)"/>
+ 	        <cylinder radius="0.025" length="$(arg anchorZ)"/>
  	      </geometry>
  	      <material name="grey">

Commit message: added possibility lo change the Y location of the first anchor that was assumed to be at 0
however, for consistency with kinematics definition of psi, both anchors
should be on the same X and Z! and only Y can be changed in the second
anchor

File: urdf/climbingrobot2.xacro (robot description, xacro)
@@ -195,5 +195,5 @@
   <!-- Anchor 2   -->
    <joint name="anchor2_position" type="fixed">
-        <origin rpy="0 0 0" xyz="0 $(arg anchor2Y) 0"/>
+        <origin rpy="0 0 0" xyz="0 ${$(arg anchor2Y)-$(arg anchorY)} 0"/>
         <parent link="anchor"/>
         <child link="anchor_2"/>

File: urdf/climbingrobot2landing.xacro (robot description, xacro)
@@ -197,5 +197,5 @@
   <!-- Anchor 2   -->
    <joint name="anchor2_position" type="fixed">
-        <origin rpy="0 0 0" xyz="0 $(arg anchor2Y) 0"/>
+        <origin rpy="0 0 0" xyz="0 ${$(arg anchor2Y)-$(arg anchorY)} 0"/>
         <parent link="anchor"/>
         <child link="anchor_2"/>

Commit message: added double propeller

File: urdf/climbingrobot2.xacro (robot description, xacro)
@@ -13,4 +13,5 @@
    <xacro:arg name="hoist_distance" default="0.1"/>
    <xacro:arg name="hoist_base_distanceZ" default="0.05"/>
+   <xacro:arg name="double_propeller" default="false"/>
     <xacro:include filename="$(find climbingrobot_description)/gazebo/gazebo.urdf.xacro">
         <xacro:arg name="task_period" value="$(arg task_period)"/>
@@ -567,6 +568,11 @@
   <!-- END LOWER LEG LINK -->
   <!-- Joint between the base and the ${prefix} upper leg -->
+   <xacro:unless value="$(arg double_propeller)">
+   	<xacro:include filename="$(find climbingrobot_description)/urdf/propellers.urdf.xacro"/>
+   </xacro:unless>
+   <xacro:if value="$(arg double_propeller)">
+         <xacro:include filename="$(find climbingrobot_description)/urdf/propellers_couple.urdf.xacro"/>
+   </xacro:if>
    <xacro:include filename="$(find climbingrobot_description)/urdf/gazebo.urdf.xacro"/>
-   <xacro:include filename="$(find climbingrobot_description)/urdf/propellers.urdf.xacro"/>
    <xacro:climbingrobot_transmission/>
 </robot>

File: urdf/climbingrobot2landing.xacro (robot description, xacro)
@@ -14,4 +14,5 @@
    <xacro:arg name="hoist_base_distanceZ" default="0.05"/>
    <xacro:arg name="lowerleg_landing_length" default="0.3"/>
+    <xacro:arg name="double_propeller" default="false"/>
     <xacro:property name="WHEEL_pos" value="0.10183" />
     <xacro:include filename="$(find climbingrobot_description)/gazebo/gazebo.urdf.xacro">
@@ -815,5 +816,10 @@
   <!-- Joint between the base and the ${prefix} upper leg -->
    <xacro:include filename="$(find climbingrobot_description)/urdf/gazebo.urdf.xacro"/>
-   <xacro:include filename="$(find climbingrobot_description)/urdf/propellers.urdf.xacro"/>
+   <xacro:unless value="$(arg double_propeller)">
+   	<xacro:include filename="$(find climbingrobot_description)/urdf/propellers.urdf.xacro"/>
+   </xacro:unless>
+   <xacro:if value="$(arg double_propeller)">
+         <xacro:include filename="$(find climbingrobot_description)/urdf/propellers_couple.urdf.xacro"/>
+   </xacro:if>
    <xacro:climbingrobot_transmission/>
 </robot>

File: urdf/propellers.urdf.xacro (robot description, xacro)
@@ -17,30 +17,3 @@
     </visual>
   </link>
-  <!-- <link name="propeller_sx">
-    <visual>
-      <origin rpy="0 0 0" xyz="0 0 0"/>
-      <geometry>
-        <mesh filename="package://climbingrobot_description/meshes/propeller_simple.stl" scale="0.002 0.002 0.002"/>
-      </geometry>
-      <material name="blue">
-        <color rgba="0 1 0 1.0"/>
-      </material>
-    </visual>
-  </link>
-  <joint name="propeller_dx_location" type="fixed">
-    <parent link="base_link"/>
-    <child link="propeller_dx"/>
-    <origin rpy="0 -1.57 0" xyz="0.07 0.05 0.025"/>
-  </joint>
-  <link name="propeller_dx">
-    <visual>
-      <origin rpy="0 0 0" xyz="0 0 0"/>
-      <geometry>
-        <mesh filename="package://climbingrobot_description/meshes/propeller_simple.stl" scale="0.002 0.002 0.002"/>
-      </geometry>
-	<material name="blue">
-        <color rgba="0 1 0 1.0"/>
-      </material>
-    </visual>
-  </link> -->
 </robot>
