Commit message: removed collision from baselink in real robot mesh

File: urdf/climbingrobot2_real.xacro (robot description, xacro)
@@ -426,8 +426,7 @@
     </visual>
     <!-- LOWER LEG LINK COLLISION -->
-    <collision>
-      <origin rpy="0 0 0" xyz="0 0 0"/>
-      <geometry>
-       <!--mesh filename="package://climbingrobot_description/meshes/obj/with_foot/solo_lower_leg_left_side.obj" scale="1 1 1.5"/-->
+    <!--collision>
+      <origin rpy="0 0 0" xyz="0 0 0"/>
+      <geometry>
          <mesh filename="package://climbingrobot_description/meshes/alpine/alpine_body_rod.stl" scale="1 1 1"/>
       </geometry>
@@ -435,5 +434,5 @@
         <color rgba="0.7 0.7 0.7 0.5"/>
       </material>
-    </collision>
+    </collision-->
     <!-- Bullet specific paramters -->
     <contact>
