Commit message: changes for compatibility with Michele's framework

File: gazebo/gazebo.urdf.xacro (robot description, xacro)
@@ -13,5 +13,5 @@
 		<plugin filename="libgazebo_ros_p3d.so" name="gazebo_ros_p3d">
                         <robotNamespace>/$(arg robot_name)</robotNamespace>
-                        <bodyName>trunk</bodyName>
+                        <bodyName>base_link</bodyName>
 			<topicName>ground_truth</topicName>
 			<frameName>world</frameName>

File: urdf/climbingrobot.xacro (robot description, xacro)
@@ -1,10 +1,52 @@
 <?xml version="1.0" ?>
-<robot name="climber">
+<robot name="climbingrobot" xmlns:xacro="http://ros.org/wiki/xacro">
   <!-- This file is based on: https://atlas.is.localnet/confluence/display/AMDW/Quadruped+URDF+Files -->
-  <link name="mountain">
+    <!--- new_gazebo_version should be false by default because pinocchio needs it!-->
+    <xacro:arg name="robot_name" default="climbingrobot"/>
+    <xacro:arg name="new_gazebo_version" default="false"/>
+    <xacro:include filename="$(find climbingrobot_description)/gazebo/gazebo.urdf.xacro">
+        <xacro:arg name="task_period" value="$(arg task_period)"/>
+	<xacro:arg name="robot_name" value="$(arg robot_name)"/>
+    </xacro:include>
+    <xacro:include filename="$(find climbingrobot_description)/urdf/climbingrobot.transmission.xacro"/>
+ 	<link name="world"/>
+ 	<joint name="anchor_x_joint" type="prismatic">
+		<parent link="world"/>
+		<child link="fake_link1"/>
+		<axis xyz="1 0 0 "/>
+		<origin xyz="0 0 0" rpy="0 0 0"/>
+		<limit effort="1000" velocity="100.0" lower="-100" upper="100"/>
+	</joint>
+	<link name="fake_link1">
+	<inertial>
+	<mass value="0.00001"/>
+	<inertia ixx="5.8083e-4" ixy="0" ixz="0" iyy="3.0833e-5" iyz="0" izz="5.9083e-4"/>
+	</inertial>
+	</link>
+	<joint name="anchor_y_joint" type="prismatic">
+		<parent link="fake_link1"/>
+		<child link="fake_link2"/>
+		<axis xyz="0 1 0 "/>
+		<origin xyz="0 0 0" rpy="0 0 0"/>
+		<limit effort="1000" velocity="100.0" lower="-100" upper="100"/>
+	</joint>
+	<link name="fake_link2">
+	<inertial>
+	<mass value="0.00001"/>
+	<inertia ixx="5.8083e-4" ixy="0" ixz="0" iyy="3.0833e-5" iyz="0" izz="5.9083e-4"/>
+	</inertial>
+	</link>
+	<joint name="anchor_z_joint" type="prismatic">
+		<parent link="fake_link2"/>
+		<child link="anchor"/>
+		<axis xyz="0 0 1 "/>
+		<origin xyz="0 0 0" rpy="0 0 0"/>
+		<limit effort="1000" velocity="100.0" lower="-100" upper="100"/>
+	</joint>
+  <link name="anchor">
     <!--<visual>
       <origin rpy="0 0 0" xyz="0 0 0"/>
       <geometry>
-        <mesh filename="package://model/urdf/meshes/obj/cube.obj" scale="0.01 10.0 10.0"/>
+        <mesh filename="package://climbingrobot_description/meshes/obj/cube.obj" scale="0.01 10.0 10.0"/>
       </geometry>
       <material name="ground">
@@ -12,19 +54,20 @@
       </material>
     </visual>-->
-    <collision>
+    <!-- TODO manage wall collision-->
+    <!--collision>
       <origin rpy="0 0 0" xyz="0 0 0.0"/>
       <geometry>
         <box size="0.1 10.0 10.0"/>
       </geometry>
-    </collision>
-    <inertial>
-      <origin rpy="0 0 0" xyz="0 0 0.0"/>
-      <mass value="1000.0"/>
-      <inertia ixx="10.0" ixy="0.0" ixz="0.0" iyy="10.0" iyz="0.0" izz="10.0"/>
+    </collision-->
+    <inertial>
+      <origin rpy="0 0 0" xyz="0 0 0.0"/>
+      <mass value="1.0"/>
+      <inertia ixx="1.0" ixy="0.0" ixz="0.0" iyy="1.0" iyz="0.0" izz="1.0"/>
     </inertial>
   </link>
   <!-- Revolute pitch joint between the mountain and the wire -->
   <joint name="mountain_wire_pitch" type="revolute">
-    <parent link="mountain"/>
+    <parent link="anchor"/>
     <child link="pre-wire1"/>
     <limit effort="3" lower="-10" upper="10" velocity="1000"/>
@@ -39,5 +82,5 @@
       <origin rpy="0 0 0" xyz="0 0 0"/>
       <geometry>
-        <mesh filename="package://model/urdf/meshes/obj/cylinder.obj" scale="0.01 0.01 0.01"/>
+        <mesh filename="package://climbingrobot_description/meshes/obj/cylinder.obj" scale="0.01 0.01 0.01"/>
       </geometry>
       <material name="grey">
@@ -72,5 +115,5 @@
       <origin rpy="0 0 0" xyz="0 0 0"/>
       <geometry>
-        <mesh filename="package://model/urdf/meshes/obj/cylinder.obj" scale="0.01 0.01 0.01"/>
+        <mesh filename="package://climbingrobot_description/meshes/obj/cylinder.obj" scale="0.01 0.01 0.01"/>
       </geometry>
       <material name="grey">
@@ -102,19 +145,4 @@
   </joint>
   <link name="wire">
-    <visual>
-      <origin rpy="0 0 0" xyz="0 0 -2"/>
-      <geometry>
-        <mesh filename="package://model/urdf/meshes/obj/cylinder.obj" scale="0.01 0.01 4.0"/>
-      </geometry>
-      <material name="grey">
-        <color rgba=".7 .7 .7 .5"/>
-      </material>
-    </visual>
-    <collision>
-      <origin rpy="0 0 0" xyz="0 0 0.0"/>
-      <geometry>
-        <cylinder length="4" radius="0.01"/>
-      </geometry>
-    </collision>
     <inertial>
       <origin rpy="0 0 0" xyz="0 0 0.0"/>
@@ -130,24 +158,9 @@
     <!-- joint translates on x axis -->
     <axis xyz="0 0 1"/>
-    <origin rpy="0 0 0" xyz="0.0 0.0 -2.0"/>
+    <origin rpy="0 0 0" xyz="0.0 0.0 -1.0"/>
     <!-- pybullet simulation parameters -->
     <dynamics damping="0.0" friction="0.0"/>
   </joint>
   <link name="pre-base1">
-    <visual>
-      <origin rpy="0 0 0" xyz="0 0 0"/>
-      <geometry>
-        <mesh filename="package://model/urdf/meshes/obj/cylinder.obj" scale="0.01 0.01 0.01"/>
-      </geometry>
-      <material name="grey">
-        <color rgba=".7 .7 .7 .5"/>
-      </material>
-    </visual>
-    <collision>
-      <origin rpy="0 0 0" xyz="0 0 0.0"/>
-      <geometry>
-        <cylinder length="0.01" radius="0.01"/>
-      </geometry>
-    </collision>
     <inertial>
       <origin rpy="0 0 0" xyz="0 0 0.0"/>
@@ -168,20 +181,5 @@
   </joint>
   <link name="pre-base2">
-    <visual>
-      <origin rpy="0 0 0" xyz="0 0 0"/>
-      <geometry>
-        <mesh filename="package://model/urdf/meshes/obj/cylinder.obj" scale="0.01 0.01 0.01"/>
-      </geometry>
-      <material name="grey">
-        <color rgba=".7 .7 .7 .5"/>
-      </material>
-    </visual>
-    <collision>
-      <origin rpy="0 0 0" xyz="0 0 0.0"/>
-      <geometry>
-        <cylinder length="0.01" radius="0.01"/>
-      </geometry>
-    </collision>
-    <inertial>
+     <inertial>
       <origin rpy="0 0 0" xyz="0 0 0.0"/>
       <mass value="0.01"/>
@@ -201,19 +199,4 @@
   </joint>
   <link name="pre-base3">
-    <visual>
-      <origin rpy="0 0 0" xyz="0 0 0"/>
-      <geometry>
-        <mesh filename="package://model/urdf/meshes/obj/cylinder.obj" scale="0.01 0.01 0.01"/>
-      </geometry>
-      <material name="grey">
-        <color rgba=".7 .7 .7 .5"/>
-      </material>
-    </visual>
-    <collision>
-      <origin rpy="0 0 0" xyz="0 0 0.0"/>
-      <geometry>
-        <cylinder length="0.01" radius="0.01"/>
-      </geometry>
-    </collision>
     <inertial>
       <origin rpy="0 0 0" xyz="0 0 0.0"/>
@@ -225,5 +208,5 @@
   <joint name="wire_base_yaw" type="revolute">
     <parent link="pre-base3"/>
-    <child link="base"/>
+    <child link="base_link"/>
     <limit effort="3" lower="-10" upper="10" velocity="1000"/>
     <!-- joint rotates about z axis -->
@@ -233,5 +216,5 @@
     <dynamics damping="0.0" friction="0.0"/>
   </joint>
-  <link name="base">
+  <link name="base_link">
     <!-- BASE LINK INERTIAL -->
     <inertial>
@@ -246,5 +229,5 @@
       <origin rpy="0 0 0" xyz="0 0 0"/>
       <geometry>
-        <mesh filename="package://model/urdf/meshes/obj/with_foot/solo_body.obj" scale="1 1 1"/>
+        <mesh filename="package://climbingrobot_description/meshes/obj/with_foot/solo_body.obj" scale="1 1 1"/>
       </geometry>
       <material name="red">
@@ -256,5 +239,5 @@
       <origin rpy="0 0 0" xyz="0 0 0"/>
       <geometry>
-        <mesh filename="package://model/urdf/meshes/obj/with_foot/solo_body.obj" scale="1 1 1"/>
+        <mesh filename="package://climbingrobot_description/meshes/obj/with_foot/solo_body.obj" scale="1 1 1"/>
       </geometry>
     </collision>
@@ -268,5 +251,5 @@
   <!-- Joint between the base and the ${prefix} upper leg -->
   <joint name="hip_pitch" type="revolute">
-    <parent link="base"/>
+    <parent link="base_link"/>
     <child link="upper_link1"/>
     <limit effort="3" lower="-10" upper="10" velocity="1000"/>
@@ -288,5 +271,5 @@
       <origin rpy="0 0 0" xyz="0 0 0"/>
       <geometry>
-        <mesh filename="package://model/urdf/meshes/obj/with_foot/solo_upper_leg_left_side.obj"/>
+        <mesh filename="package://climbingrobot_description/meshes/obj/with_foot/solo_upper_leg_left_side.obj"/>
       </geometry>
       <material name="grey">
@@ -298,5 +281,5 @@
       <origin rpy="0 0 0" xyz="0 0 0"/>
       <geometry>
-        <mesh filename="package://model/urdf/meshes/obj/with_foot/solo_upper_leg_left_side.obj"/>
+        <mesh filename="package://climbingrobot_description/meshes/obj/with_foot/solo_upper_leg_left_side.obj"/>
       </geometry>
         <material name="white">
@@ -331,5 +314,5 @@
       <origin rpy="0 0 0" xyz="0 0 0"/>
       <geometry>
-        <mesh filename="package://model/urdf/meshes/obj/with_foot/solo_upper_leg_left_side.obj"/>
+        <mesh filename="package://climbingrobot_description/meshes/obj/with_foot/solo_upper_leg_left_side.obj"/>
       </geometry>
       <material name="grey">
@@ -341,5 +324,5 @@
       <origin rpy="0 0 0" xyz="0 0 0"/>
       <geometry>
-        <mesh filename="package://model/urdf/meshes/obj/with_foot/solo_upper_leg_left_side.obj"/>
+        <mesh filename="package://climbingrobot_description/meshes/obj/with_foot/solo_upper_leg_left_side.obj"/>
       </geometry>
         <material name="white">
@@ -376,5 +359,5 @@
       <origin rpy="0 0 0" xyz="0 0 0"/>
       <geometry>
-        <mesh filename="package://model/urdf/meshes/obj/with_foot/solo_lower_leg_left_side.obj" scale="1 1 1.5"/>
+        <mesh filename="package://climbingrobot_description/meshes/obj/with_foot/solo_lower_leg_left_side.obj" scale="1 1 1.5"/>
       </geometry>
         <material name="white">
@@ -386,5 +369,5 @@
       <origin rpy="0 0 0" xyz="0 0 0"/>
       <geometry>
-        <mesh filename="package://model/urdf/meshes/obj/with_foot/solo_lower_leg_left_side.obj"/>
+        <mesh filename="package://climbingrobot_description/meshes/obj/with_foot/solo_lower_leg_left_side.obj"/>
       </geometry>
       <material name="grey">
@@ -421,5 +404,5 @@
       <origin rpy="0 0 0" xyz="0 0 0"/>
       <geometry>
-        <mesh filename="package://model/urdf/meshes/obj/with_foot/solo_foot.obj"/>
+        <mesh filename="package://climbingrobot_description/meshes/obj/with_foot/solo_foot.obj"/>
       </geometry>
 	<material name="black">
@@ -431,5 +414,5 @@
       <origin rpy="0 0 0" xyz="0 0 0"/>
       <geometry>
-        <mesh filename="package://model/urdf/meshes/obj/with_foot/solo_foot.obj"/>
+        <mesh filename="package://climbingrobot_description/meshes/obj/with_foot/solo_foot.obj"/>
       </geometry>
       <material name="grey">
@@ -445,3 +428,4 @@
   <!-- END LOWER LEG LINK -->
   <!-- Joint between the base and the ${prefix} upper leg -->
+   <xacro:climbingrobot_transmission/>
 </robot>

Commit message: adjusting base link mass such that the overall robot mass is 5 kg

File: gazebo/gazebo.urdf.xacro (robot description, xacro)
@@ -1,6 +1,6 @@
 <?xml version="1.0"?>
 <robot xmlns:xacro="http://ros.org/wiki/xacro">
-<xacro:arg name="task_period" default="0.004" />
-<xacro:arg name="robot_name" default="starbot" />
+<xacro:arg name="task_period" default="0.001" />
+<xacro:arg name="robot_name" default="climbingrobot" />
 	<gazebo>
 		<plugin name="gazebo_ros_controller_manager" filename="libgazebo_ros_control.so">

File: urdf/climbingrobot.xacro (robot description, xacro)
@@ -150,5 +150,5 @@
       <origin rpy="0 0 0" xyz="0 0 0"/>
       <!-- <mass value="0.36"/> -->
-      <mass value="5.0"/>
+      <mass value="3.47"/>
       <!-- The base is extremely symmetrical. -->
       <inertia ixx="0.5" ixy="0.0" ixz="0.0" iyy="0.5" iyz="0.0" izz="0.5"/>
